File: PSEC5_Ctrl_Board/_autosave-PSEC5_Ctrl_Board.kicad_sch (KiCad schematic)
At the start: 3 parts, among them J3 ADM6-60-01.5-L-4-2-A-TR, J4 ADM6-60-01.5-L-4-2-A-TR, J5 QSH-040-01-X-D-DP-A

Commit message: A lil more to ctlrbrd, more to come very soon
Parts:
- added J9: QSH-040-01-X-D-DP-A, QSH-040-01-X-D-DP-A:SAMTEC_QSH-040-01-X-D-DP-A, symbol PSEC5_ctrlbd:QSH-040-01-X-D-DP-A
Connections:
- net CLKOUT: no longer J5.23
- net DISCBIAS: now also J5.39; no longer J4.B39, J5.24
- net GND: now also J9.G1 (GND_S1), J9.G2 (GND_S1__1), J9.G3 (GND_S1__2), J9.G4 (GND_S1__3)
- net PICO: now also J9.11; no longer J4.B16, J5.33
- net POCI: now also J9.09; no longer J5.03
- net READBIAS1: now also J5.33; no longer J4.B34, J5.18
- net READBIAS2: now also J5.35; no longer J4.B36, J5.20
- net READOUT1: no longer J5.05
- net READOUT2: no longer J5.07
- net READOUT3: no longer J5.09
- net READOUT4: no longer J5.11
- net READOUT5: no longer J5.13
- net READOUT6: no longer J5.15
- net READOUT7: no longer J5.17
- net READOUT8: no longer J5.19
- net REFCLKOUT: no longer J5.25
- net THRES1: now also J5.01; no longer J4.B22, J5.02
- net THRES2: now also J5.03; no longer J4.B24, J5.04
- net THRES3: now also J5.05; no longer J4.B25, J5.06
- net THRES4: now also J5.07; no longer J4.B27, J5.08
- net THRES5: now also J5.09; no longer J4.B28, J5.10
- net THRES6: now also J5.11; no longer J4.B30, J5.12
- net THRES7: now also J5.13; no longer J4.B31, J5.14
- net THRES8: now also J5.15; no longer J4.B33, J5.16
- net TRIGGEROUT: no longer J5.21
- net WBUFBIAS: now also J5.37; no longer J4.B37, J5.22
- net prep_VTUNE: no longer J5.01
- net READCLK: no longer names the net of J4.B12
- net READCLK: no longer J5.27
- net RESET: no longer names the net of J4.B18
- net RESET: no longer J5.35
- net SIGNAL1: no longer names the net of J4.B40
- net SIGNAL1: no longer J5.26
- net SIGNAL2: no longer names the net of J4.B44
- net SIGNAL2: no longer J5.28
- net SIGNAL3: no longer names the net of J4.B45
- net SIGNAL3: no longer J5.30
- net SIGNAL4: no longer names the net of J4.B46
- net SIGNAL4: no longer J5.32
- net SIGNAL5: no longer names the net of J4.B48
- net SIGNAL5: no longer J5.34
- net SIGNAL6: no longer names the net of J4.B49
- net SIGNAL6: no longer J5.36
- net SIGNAL7 renamed SIGNAL8+
- net SIGNAL8: no longer names the net of J4.B52
- net SIGNAL8: no longer J5.40
- net SIGNAl7: no longer names the net of J4.B50
- net SPICLK: no longer names the net of J4.B19
- net SPICLK: no longer J5.37
- net TRIGGERIN: no longer names the net of J4.B13
- net TRIGGERIN: no longer J5.29
- net VCOCTRL: no longer names the net of J4.B15
- net VCOCTRL: no longer J5.31
- net postp_VTUNE: no longer names the net of J4.B21
- net postp_VTUNE: no longer J5.39
- new net 1V2: J9.02
- new net 1V8: J9.04
- new net 2V5: J9.06
- new net 3V3: J9.08
- new net 5V: J9.10
- new net ADC_SCLK: J9.29
- new net ADC_SDO: J9.33
- new net DAC_SCLK: J9.21
- new net DAC_V_IN: J9.27
- new net OscRefClk: J9.01
- new net Psec5RST: J9.15
- new net Psec5ReadClk: J9.17
- new net Psec5RefClk: J9.03
- new net Psec5TriggerIn: J9.07
- new net Psec5TriggerOut: J9.05
- new net SIGNAL1+: J5.02
- new net SIGNAL1-: J5.04
- new net SIGNAL2+: J5.06
- new net SIGNAL2-: J5.08
- new net SIGNAL3+: J5.10
- new net SIGNAL3-: J5.12
- new net SIGNAL4+: J5.14
- new net SIGNAL4-: J5.16
- new net SIGNAL5+: J5.26
- new net SIGNAL5-: J5.28
- new net SIGNAL6+: J5.30
- new net SIGNAL6-: J5.32
- new net SIGNAL7+: J5.34
- new net SIGNAL7-: J5.36
- new net SIGNAL8-: J5.40
- new net SPIClk: J9.13
- new net SYNC_N: J9.25
Other:
- added sheet adcdac (adccad.kicad_sch)
- added sheet samtectest (samtectest.kicad_sch)
- sheet JTAG ports: added CLK, RST, TDI, TDO, TMS; removed none
- sheet Peripherals_Ctrl ports: added ADC_1.8AVDD, ADC_1.8DVDD, ADC_CLK+, ADC_CLK-, ADC_DOUT1+, ADC_DOUT1-, ADC_DOUT2+, ADC_DOUT2-, ADC_DOUT3+, ADC_DOUT3-, ADC_DOUT4+, ADC_DOUT4-, ADC_DOUT5+, ADC_DOUT5-, ADC_DOUT6+, ADC_DOUT6-, ADC_DOUT7+, ADC_DOUT7-, ADC_DOUT8+, ADC_DOUT8-, ADC_VREF, DCO+, DCO-, FCO+, FCO-, READOUT1+, READOUT1-, READOUT2+, READOUT2-, READOUT3+, READOUT3-, READOUT4+, READOUT4-, READOUT5+, READOUT5-, READOUT6+, READOUT6-, READOUT7+, READOUT7-, READOUT8+, READOUT8-; removed none
- sheet SDcard ports: added SD_CLK, SD_CMD, SD_DAT0, SD_DAT1, SD_DAT2, SD_DAT3, SD_DETECT, SD_PWR_EN, SD_SEL; removed none
- note added: "ANALOG SAMTEC"
- note added: "DIGITAL SAMTEC + OTHER"
- note removed: "INPUTS"
- note removed: "OUTPUTS"
- moved on the sheet: J3A, J4A
