File: PSEC5_Ctrl_Board/samtectest.kicad_sch (KiCad schematic)
At the start: 2 parts, among them J10 QSH-040-01-X-D-DP-A, J11 QSH-040-01-X-D-DP-A

Commit message: Large Updates, Touching up before further aproval
Parts:
- removed J10, J11: QSH-040-01-X-D-DP-A, QSH-040-01-X-D-DP-A:SAMTEC_QSH-040-01-X-D-DP-A, symbol PSEC5_ctrlbd:QSH-040-01-X-D-DP-A
Other:
- note added: "NOTE: 1.5 Connector is the Connector that will lay on the Control board. The 3.5 connector goes on the bottom of the Kria Module"
- note removed: "ANALOG SAMTEC"
- note removed: "DIGITAL SAMTEC + OTHER"
- title: (none) -> SOM240_1
