File: PSEC5_Ctrl_Board/adccad.kicad_sch (KiCad schematic)
At the start: 10 parts, among them U2 LTC2600CGN_PBF, U4 LTC2600CGN_PBF

Commit message: Minor Schematic Changes, ERC still haunts me :(
Parts:
- removed TP19: SDO1, symbol Connector:TestPoint
Connections:
- net SDI_DAC_BIAS: no longer U4.9 (SDI)
- net at U2.10 (SDO): now also U4.9 (SDI)
- net 1V8_DUT renamed 1V8_IO
- net 3V3_DUT renamed 3V3_IO
- net CS/LD_DAC* renamed CS/LD_DAC1*
- net CS/LD_DAC1*: no longer U4.7 (*CS/LD)
- new net CS/LD_DAC2*: U4.7 (*CS/LD)
- no-connect marks 4 -> 5
Changed lines of the file:
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@@
+	)
+	(no_connect
+		(at 54.61 43.18)
 	)
 	(no_connect
@@
 	(wire
 		(pts
+			(xy 69.85 35.56) (xy 53.34 35.56)
+		)
+		(stroke
+			(width 0)
+			(type default)
+		)
+	)
+	(wire
+		(pts
+			(xy 215.9 74.93) (xy 242.57 74.93)
+		)
+		(stroke
+			(width 0)
+			(type default)
+		)
+	)
+	(wire
+		(pts
 			(xy 69.85 31.75) (xy 53.34 31.75)
 		)
@@
 	(wire
 		(pts
-			(xy 215.9 74.93) (xy 242.57 74.93)
-		)
-		(stroke
-			(width 0)
-			(type default)
-		)
-	)
-	(wire
-		(pts
 			(xy 220.98 148.59) (xy 220.98 158.75)
 		)
@@
 	(wire
 		(pts
-			(xy 215.9 151.13) (xy 240.03 151.13)
-		)
-		(stroke
-			(width 0)
-			(type default)
-		)
-	)
-	(wire
-		(pts
 			(xy 149.86 133.35) (xy 106.68 133.35)
 		)
@@
 	(wire
 		(pts
+			(xy 53.34 43.18) (xy 54.61 43.18)
+		)
+		(stroke
+			(width 0)
+			(type default)
+		)
+	)
+	(wire
+		(pts
 			(xy 106.68 133.35) (xy 106.68 134.62)
 		)
@@
 	(wire
 		(pts
+			(xy 218.44 151.13) (xy 215.9 151.13)
+		)
+		(stroke
+			(width 0)
+			(type default)
+		)
+	)
+	(wire
+		(pts
 			(xy 125.73 138.43) (xy 149.86 138.43)
 		)
@@
 	(wire
 		(pts
+			(xy 218.44 77.47) (xy 218.44 151.13)
+		)
+		(stroke
+			(width 0)
+			(type default)
+		)
+	)
+	(wire
+		(pts
 			(xy 241.3 133.35) (xy 246.38 133.35)
 		)
@@
 	(wire
 		(pts
-			(xy 218.44 77.47) (xy 218.44 86.36)
-		)
-		(stroke
-			(width 0)
-			(type default)
-		)
-	)
-	(wire
-		(pts
 			(xy 115.57 146.05) (xy 115.57 148.59)
 		)
@@
 	(wire
 		(pts
-			(xy 53.34 39.37) (xy 69.85 39.37)
-		)
-		(stroke
-			(width 0)
-			(type default)
-		)
-	)
-	(wire
-		(pts
 			(xy 127 69.85) (xy 149.86 69.85)
 		)
@@
 	(wire
 		(pts
-			(xy 69.85 35.56) (xy 53.34 35.56)
+			(xy 69.85 39.37) (xy 53.34 39.37)
 		)
 		(stroke
@@
 	)
 	(label "CLR_DAC*"
-		(at 69.85 31.75 180)
+		(at 69.85 35.56 180)
 		(fields_autoplaced yes)
 		(effects
@@
 	)
 	(label "SCK_DAC"
-		(at 69.85 35.56 180)
+		(at 69.85 39.37 180)
 		(fields_autoplaced yes)
 		(effects
@@
 		)
 	)
-	(label "CS{slash}LD_DAC*"
+	(label "CS{slash}LD_DAC1*"
 		(at 69.85 27.94 180)
 		(fields_autoplaced yes)
@@
 		)
 	)
-	(label "SDI_DAC_BIAS"
-		(at 69.85 39.37 180)
-		(fields_autoplaced yes)
-		(effects
-			(font
-				(size 1.27 1.27)
-			)
-			(justify right bottom)
-		)
-	)
 	(label "DAC_THRES3_OUT"
 		(at 127 69.85 0)
@@
 		)
 	)
-	(label "CS{slash}LD_DAC*"
+	(label "CS{slash}LD_DAC2*"
 		(at 125.73 148.59 0)
 		(fields_autoplaced yes)
@@
 		)
 	)
-	(label "SDI_DAC_BIAS"
-		(at 240.03 151.13 180)
-		(fields_autoplaced yes)
-		(effects
-			(font
-				(size 1.27 1.27)
-			)
-			(justify right bottom)
-		)
-	)
 	(label "DAC_THRES7_OUT"
 		(at 58.42 83.82 0)
@@
 		)
 	)
+	(label "CS{slash}LD_DAC2*"
+		(at 69.85 31.75 180)
+		(fields_autoplaced yes)
+		(effects
+			(font
+				(size 1.27 1.27)
+			)
+			(justify right bottom)
+		)
+	)
 	(label "SDI_DAC_THRES"
 		(at 238.76 80.01 180)
@@
 		)
 	)
-	(label "CS{slash}LD_DAC*"
+	(label "CS{slash}LD_DAC1*"
 		(at 127 77.47 0)
 		(fields_autoplaced yes)
@@
 		)
 	)
-	(global_label "3V3_DUT"
+	(global_label "3V3_IO"
 		(shape input)
 		(at 228.6 129.54 90)
@@
 		)
 		(property "Intersheetrefs" "${INTERSHEET_REFS}"
-			(at 228.6 118.5115 90)
+			(at 228.6 120.1443 90)
 			(effects
 				(font
@@
 		)
 	)
-	(global_label "1V8_DUT"
+	(global_label "1V8_IO"
 		(shape input)
 		(at 113.03 74.93 180)
@@
 		)
 		(property "Intersheetrefs" "${INTERSHEET_REFS}"
-			(at 102.0015 74.93 0)
+			(at 103.6343 74.93 0)
 			(effects
 				(font
@@
 		)
 	)
-	(global_label "3V3_DUT"
+	(global_label "3V3_IO"
 		(shape input)
 		(at 228.6 58.42 90)
@@
 		)
 		(property "Intersheetrefs" "${INTERSHEET_REFS}"
-			(at 228.6 47.3915 90)
+			(at 228.6 49.0243 90)
 			(effects
 				(font
@@
 		)
 	)
-	(global_label "1V8_DUT"
+	(global_label "1V8_IO"
 		(shape input)
 		(at 104.14 146.05 180)
@@
 		)
 		(property "Intersheetrefs" "${INTERSHEET_REFS}"
-			(at 93.1115 146.05 0)
+			(at 94.7443 146.05 0)
 			(effects
 				(font
@@
 		)
 	)
-	(hierarchical_label "CS{slash}LD_DAC*"
+	(hierarchical_label "CS{slash}LD_DAC1*"
 		(shape input)
 		(at 53.34 27.94 180)
@@
 	(hierarchical_label "SCK_DAC"
 		(shape input)
+		(at 53.34 39.37 180)
+		(fields_autoplaced yes)
+		(effects
+			(font
+				(size 1.27 1.27)
+			)
+			(justify right)
+		)
+	)
+	(hierarchical_label "CLR_DAC*"
+		(shape input)
 		(at 53.34 35.56 180)
 		(fields_autoplaced yes)
@@
 		)
 	)
-	(hierarchical_label "CLR_DAC*"
+	(hierarchical_label "CS{slash}LD_DAC2*"
 		(shape input)
 		(at 53.34 31.75 180)
@@
 	(hierarchical_label "SDI_DAC_BIAS"
 		(shape input)
-		(at 53.34 39.37 180)
-		(fields_autoplaced yes)
-		(effects
-			(font
-				(size 1.27 1.27)
-			)
-			(justify right)
-		)
-	)
-	(symbol
-		(lib_id "Connector:TestPoint")
-		(at 218.44 86.36 270)
-		(unit 1)
-		(exclude_from_sim no)
-		(in_bom yes)
-		(on_board yes)
-		(dnp no)
-		(fields_autoplaced yes)
-		(property "Reference" "TP19"
-			(at 223.52 85.0899 90)
-			(effects
-				(font
-					(size 1.27 1.27)
-				)
-				(justify left)
-			)
-		)
-		(property "Value" "SDO1"
-			(at 223.52 87.6299 90)
-			(effects
-				(font
-					(size 1.27 1.27)
-				)
-				(justify left)
-			)
-		)
-		(property "Footprint" ""
-			(at 218.44 91.44 0)
-			(effects
-				(font
-					(size 1.27 1.27)
-				)
-				(hide yes)
-			)
-		)
-		(property "Datasheet" "~"
-			(at 218.44 91.44 0)
-			(effects
-				(font
-					(size 1.27 1.27)
-				)
-				(hide yes)
-			)
-		)
-		(property "Description" "test point"
-			(at 218.44 86.36 0)
-			(effects
-				(font
-					(size 1.27 1.27)
-				)
-				(hide yes)
-			)
-		)
-		(pin "1"
-		)
-		(instances
-			(project ""
-				(path "/165f2ae6-d522-4adf-a6c4-bb137b209d33/1f6d7a03-cfad-4370-8d2b-49ab19e248d8/9bd9ffce-acff-4ff9-8380-cb9ceb30e6db"
-					(reference "TP19")
-					(unit 1)
-				)
-			)
-		)
-	)
+		(at 53.34 43.18 180)
+		(fields_autoplaced yes)
+		(effects
+			(font
+				(size 1.27 1.27)
+			)
+			(justify right)
+		)
+	)

Commit message: Some more Changes
Parts:
- added TP19: SDO2, symbol Connector:TestPoint
Connections:
- net SDI_DAC_BIAS: now also U4.9 (SDI)
- net at U2.10 (SDO): now also TP19.1; no longer U4.9 (SDI)
- net SCK_DAC renamed SCK_DAC1
- net SCK_DAC1: no longer U4.8 (SCK)
- new net SCK_DAC2: U4.8 (SCK)
- no-connect marks 5 -> 4
Other:
- note removed: "Currently, both DAC's have the following pins shorted:* *CS/LD* SCK *CLR However, the SDI pins are independent of eachother"

Commit message: ERC "Done" (4 errors left) Schematic "Done"
Parts:
- added C29, C31: 0.1u, Capacitor_SMD:C_0603_1608Metric, symbol Device:C_Small
- added C30, C32: 1n, Capacitor_SMD:C_0603_1608Metric, symbol Device:C_Small
- added U7, U8: MCP1501-25E/SN, SOIC8_NARROW_SN_MCH, symbol PSEC5_ctrlbd:MCP1501-25E_SN
Connections:
- net 3V3_IO: now also C29.1, C31.1, U7.1 (VDD), U7.3 (*SHDN), U8.1 (VDD), U8.3 (*SHDN); no longer C91.1, C92.1, U2.16 (VCC), U4.16 (VCC)
- net GND: now also C29.2, C30.2, C31.2, C32.2, U7.2 (GND), U7.4 (GND), U7.5 (GND), U7.6 (GND), U8.2 (GND), U8.4 (GND), U8.5 (GND), U8.6 (GND)
- net 1V8_IO: no longer names the net of C90.1, U2.6 (REF)
- net 1V8_IO: now also C30.1, U7.7 (OUT), U7.8 (FEEDBACK); no longer C89.1, U4.6 (REF)
- new net: C32.1, C89.1, U4.6 (REF), U8.7 (OUT), U8.8 (FEEDBACK)
- new net 2V5_IO: C91.1, C92.1, U2.16 (VCC), U4.16 (VCC)
Other:
- note added: "NOTE: DAC will run at 3V5"
- note removed: "NOTE: DAC will run at 3V3"
- moved on the sheet: C89, C90, C91, C92, R72, R77, TP19, TP20, U2, U4
