File: PSEC5_Ctrl_Board/PSEC5_Ctrl_Board.kicad_pcb (KiCad board)
At the start: 10 copper layers, 170 x 125.7 mm, 278 parts, among them J1 1766343, J10 ADM6-60-01.5-L-4-2-A-TR, J12 878311420, J14 ZX62D-B-5P830, J2 QSH-040-01-X-D-DP-A, J4 QSH-040-01-X-D-DP-A, J5 ADM6-60-01.5-L-4-2-A-TR (1), J6 1040310811, J9 1766343, Q4 NMOS, Q6 NMOS, Q8 NMOS, SW1 SW_MEC_5G, SW2 SW_MEC_5G, T2 7499111446, U1 88E1512-A0-NNP2C000, U10 PUSB3FR4Z, U11 TPS3808G01QDRVRQ1, U12 TPS3808G01QDRVRQ1, U14 SIA427ADJ-T1-GE3, U16 OKX-T/5-D12N-C, U2 LTC2600CGN_PBF, U3 PUSB3FR4Z, U4 LTC2600CGN_PBF, U5 OKX-T/5-D12N-C, U6 PI4ULS3V4857GEAEX, U7 MCP1501-25E/SN, U8 MCP1501-25E/SN, U9 FT230XQ-R, Y3 ASE2-25.000MHZ-ET

Commit message: Small Additions
Parts:
- removed T2: 7499111446, Connector_RJ:RJ45_Wuerth_7499111446_Horizontal
- added J3: ADM6-60-01.5-L-4-2-A-TR, ADM6_60_01_5_L_4_2_A_TR (1):SAMTEC_ADM6-60-01.5-L-4-2-A-TR, F.Cu at (21.7, 3.20)
- added T1: 7499111446, Connector_RJ:RJ45_Wuerth_7499111446_Horizontal, F.Cu at (58.5, -34.8)
- U7: moved to B.Cu
- moved U7 99.0 mm to (207.0, 52.1)
- moved U2 79.8 mm to (216.2, 52.1)
- moved R51 64.0 mm to (218.4, 66.3), turned to -90 degrees
- moved C76 56.4 mm to (232.7, 72.6), turned to -90 degrees
- moved C77 53.5 mm to (234.2, 72.6), turned to -90 degrees
- moved C11 53.3 mm to (217.9, 72.4), turned to -90 degrees
- moved R62 52.5 mm to (218.4, 69.3), turned to -90 degrees
- moved C80 51.4 mm to (236.7, 73.9), turned to -90 degrees
- moved C16 50.1 mm to (221.2, 73.4), turned to -90 degrees
- moved R16 49.7 mm to (239.5, 66.5), turned to -90 degrees
- moved R17 48.1 mm to (238.0, 66.5), turned to -90 degrees
- moved ADC1 47.9 mm to (236.2, 80.9)
- moved C81 47.7 mm to (238.5, 73.2), turned to -90 degrees
- moved R48 47.4 mm to (223.5, 66.6), turned to -90 degrees
- moved R50 47.1 mm to (220.0, 66.3), turned to -90 degrees
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Connections:
- 1M2 pad 2: 3V3_IO -> GND
- ADC1 pad 11: 1V2_Banks -> GND
- ADC1 pad 26: 1V2_Banks -> GND
- ADC1 pad 30: 1V2_Banks -> GND
- ADC1 pad 31: 1V2_Banks -> GND
- ADC1 pad 41: 1V2_Banks -> GND
- ADC1 pad 49: 1V2_Banks -> GND
- ADC2 pad 11: 1V2_Banks -> GND
- ADC2 pad 26: 1V2_Banks -> GND
- ADC2 pad 30: 1V2_Banks -> GND
- ADC2 pad 31: 1V2_Banks -> GND
- ADC2 pad 41: 1V2_Banks -> GND
- ADC2 pad 49: 1V2_Banks -> GND
- C1 pad 2: 1V2_Banks -> GND
- C10 pad 2: 1V2_Banks -> GND
- C106 pad 2: 3V3_IO -> GND
- C107 pad 2: 1V2_Banks -> GND
- C109 pad 2: 1V2_Banks -> GND
- C11 pad 2: 1V2_Banks -> GND
- C110 pad 2: 1V2_Banks -> GND
- C111 pad 2: 1V2_Banks -> GND
- C112 pad 2: 1V2_Banks -> GND
- C113 pad 2: 1V2_Banks -> GND
- C114 pad 2: 1V2_Banks -> GND
- C115 pad 2: 1V2_Banks -> GND
- C116 pad 2: 1V2_Banks -> GND
- C117 pad 2: 1V2_Banks -> GND
- C118 pad 2: 3V3_IO -> GND
- C119 pad 2: 3V3_IO -> GND
- C12 pad 2: 1V2_Banks -> GND
- C13 pad 2: 1V2_Banks -> GND
- C14 pad 2: 1V2_Banks -> GND
- C15 pad 2: 1V2_Banks -> GND
- C16 pad 2: 1V2_Banks -> GND
- C17 pad 2: 3V3_IO -> GND
- C18 pad 2: 1V2_Banks -> GND
- C19 pad 2: 1V2_Banks -> GND
- C2 pad 2: 1V2_Banks -> GND
- C20 pad 2: 1V2_Banks -> GND
- C21 pad 2: 3V3_IO -> GND
- C22 pad 2: 1V2_Banks -> GND
- C23 pad 2: 1V2_Banks -> GND
- C25 pad 2: 1V2_Banks -> GND
- C26 pad 2: 1V2_Banks -> GND
- C27 pad 2: 1V2_Banks -> GND
- C28 pad 2: 1V2_Banks -> GND
- C29 pad 2: 1V2_Banks -> GND
- C3 pad 2: 1V2_Banks -> GND
- C30 pad 2: 1V2_Banks -> GND
- C31 pad 2: 1V2_Banks -> GND
- C32 pad 2: 1V2_Banks -> GND
- C33 pad 2: 1V2_Banks -> GND
- C34 pad 2: 1V2_Banks -> GND
- C37 pad 2: 1V2_Banks -> GND
- C38 pad 2: 1V2_Banks -> GND
- C4 pad 2: 1V2_Banks -> GND
- C41 pad 2: 1V2_Banks -> GND
- C42 pad 2: 1V2_Banks -> GND
- C43 pad 2: 1V2_Banks -> GND
- C44 pad 2: 1V2_Banks -> GND
- C45 pad 2: 1V2_Banks -> GND
- C46 pad 2: 3V3_IO -> GND
- C47 pad 2: 1V2_Banks -> GND
- C48 pad 2: 3V3_IO -> GND
- C49 pad 2: 3V3_IO -> GND
- C50 pad 2: 3V3_IO -> GND
- C51 pad 2: 3V3_IO -> GND
- C52 pad 2: 3V3_IO -> GND
- C53 pad 2: 3V3_IO -> GND
- C54 pad 2: 3V3_IO -> GND
- C55 pad 2: 3V3_IO -> GND
- C56 pad 2: 3V3_IO -> GND
- C57 pad 2: 3V3_IO -> GND
- C58 pad 2: 3V3_IO -> GND
- C59 pad 2: 3V3_IO -> GND
- C6 pad 2: 1V2_Banks -> GND
- C60 pad 2: 3V3_IO -> GND
- C61 pad 2: 3V3_IO -> GND
- C62 pad 2: 3V3_IO -> GND
- C63 pad 2: 3V3_IO -> GND
- C64 pad 2: 3V3_IO -> GND
- C65 pad 2: 1V2_Banks -> GND
- C66 pad 2: 1V2_Banks -> GND
- C67 pad 2: 1V2_Banks -> GND
- C68 pad 2: 1V2_Banks -> GND
- C69 pad 2: 1V2_Banks -> GND
- C7 pad 2: 1V2_Banks -> GND
- C70 pad 2: 1V2_Banks -> GND
- C71 pad 2: 1V2_Banks -> GND
- C72 pad 2: 1V2_Banks -> GND
- C73 pad 2: 1V2_Banks -> GND
- C74 pad 2: 1V2_Banks -> GND
- C75 pad 2: 1V2_Banks -> GND
- C76 pad 2: 1V2_Banks -> GND
- C77 pad 2: 1V2_Banks -> GND
- C78 pad 2: 1V2_Banks -> GND
- C79 pad 2: 1V2_Banks -> GND
- C8 pad 2: 1V2_Banks -> GND
- C80 pad 2: 1V2_Banks -> GND
- C81 pad 2: 1V2_Banks -> GND
- C82 pad 2: 1V2_Banks -> GND
- C83 pad 1: 1V2_Banks -> 1V8_Banks
- C83 pad 2: 1V2_Banks -> GND
- C84 pad 1: 1V2_Banks -> 1V8_Banks
- C84 pad 2: 1V2_Banks -> GND
- C85 pad 2: 1V2_Banks -> GND
- C86 pad 1: 1V2_Banks -> 1V8_Banks
- C86 pad 2: 1V2_Banks -> GND
- C87 pad 1: 1V2_Banks -> 1V8_Banks
- C87 pad 2: 1V2_Banks -> GND
- C88 pad 2: 1V2_Banks -> GND
- C89 pad 2: 1V2_Banks -> GND
- C9 pad 2: 1V2_Banks -> GND
- C90 pad 2: 1V2_Banks -> GND
- C91 pad 2: 1V2_Banks -> GND
- C92 pad 2: 1V2_Banks -> GND
- C93 pad 2: 1V2_Banks -> GND
- C94 pad 2: 1V2_Banks -> GND
- C95 pad 2: 1V2_Banks -> GND
- C96 pad 2: 1V2_Banks -> GND
- C97 pad 2: 1V2_Banks -> GND
- C98 pad 2: 1V2_Banks -> GND
- J10 pad A01: 1V2_Banks -> GND
- J10 pad A02: 1V2_Banks -> GND
- J10 pad A05: 1V2_Banks -> GND
- J10 pad A08: 1V2_Banks -> GND
- J10 pad A11: 1V2_Banks -> GND
- J10 pad A14: 1V2_Banks -> GND
- J10 pad A18: 1V2_Banks -> GND
- J10 pad A21: 1V2_Banks -> GND
- J10 pad A26: 1V2_Banks -> GND
- J10 pad A33: 1V2_Banks -> GND
- J10 pad A37: 1V2_Banks -> GND
- J10 pad A41: 1V2_Banks -> GND
- J10 pad A45: 1V2_Banks -> GND
- J10 pad A46: 1V2_Banks -> GND
- J10 pad A49: 1V2_Banks -> GND
- J10 pad A50: 1V2_Banks -> GND
- J10 pad A53: 1V2_Banks -> GND
- J10 pad A54: 1V2_Banks -> GND
- J10 pad A57: 1V2_Banks -> GND
- J10 pad A58: 1V2_Banks -> GND
- J10 pad B03: 1V2_Banks -> GND
- J10 pad B06: 1V2_Banks -> GND
- J10 pad B09: 1V2_Banks -> GND
- J10 pad B12: 1V2_Banks -> GND
- J10 pad B15: 1V2_Banks -> GND
- J10 pad B19: 1V2_Banks -> GND
- J10 pad B23: 1V2_Banks -> GND
- J10 pad B27: 1V2_Banks -> GND
- J10 pad B31: 1V2_Banks -> GND
- J10 pad B35: 1V2_Banks -> GND
- J10 pad B39: 1V2_Banks -> GND
- J10 pad B43: 1V2_Banks -> GND
- J10 pad B47: 1V2_Banks -> GND
- J10 pad B48: 1V2_Banks -> GND
- J10 pad B51: 1V2_Banks -> GND
- J10 pad B52: 1V2_Banks -> GND
- J10 pad B55: 1V2_Banks -> GND
- J10 pad B56: 1V2_Banks -> GND
- J10 pad B59: 1V2_Banks -> GND
- J12 pad 1: 1V2_Banks -> GND
- J12 pad 11: 1V2_Banks -> GND
- J12 pad 13: 1V2_Banks -> GND
- J12 pad 3: 1V2_Banks -> GND
- J12 pad 5: 1V2_Banks -> GND
- J12 pad 7: 1V2_Banks -> GND
- J12 pad 9: 1V2_Banks -> GND
- J14 pad 5: 1V2_Banks -> GND
- J2 pad G1: 1V2_Banks -> GND
- J2 pad G2: 1V2_Banks -> GND
- J2 pad G3: 1V2_Banks -> GND
- J2 pad G4: 1V2_Banks -> GND
- J2 pad G5: 1V2_Banks -> GND
- J2 pad G6: 1V2_Banks -> GND
- J2 pad G7: 1V2_Banks -> GND
- J2 pad G8: 1V2_Banks -> GND
- J4 pad G1: 1V2_Banks -> GND
- J4 pad G2: 1V2_Banks -> GND
- J4 pad G3: 1V2_Banks -> GND
- J4 pad G4: 1V2_Banks -> GND
- J4 pad G5: 1V2_Banks -> GND
- J4 pad G6: 1V2_Banks -> GND
- J4 pad G7: 1V2_Banks -> GND
- J4 pad G8: 1V2_Banks -> GND
- J5 pad A01: 1V2_Banks -> GND
- J5 pad A02: 1V2_Banks -> GND
- J5 pad A05: 1V2_Banks -> GND
- J5 pad A06: 1V2_Banks -> GND
- J5 pad A09: 1V2_Banks -> GND
- J5 pad A10: 1V2_Banks -> GND
- J5 pad A13: 1V2_Banks -> GND
- J5 pad A16: 1V2_Banks -> GND
- J5 pad A19: 1V2_Banks -> GND
- J5 pad A22: 1V2_Banks -> GND
- J5 pad A25: 1V2_Banks -> GND
- J5 pad A28: 1V2_Banks -> GND
- J5 pad A31: 1V2_Banks -> GND
- J5 pad A34: 1V2_Banks -> GND
- J5 pad A37: 1V2_Banks -> GND
- J5 pad A40: 1V2_Banks -> GND
- J5 pad A43: 1V2_Banks -> GND
- J5 pad A44: 1V2_Banks -> 1V8_Banks
- J5 pad A45: 1V2_Banks -> GND
- J5 pad A49: 1V2_Banks -> GND
- J5 pad A53: 1V2_Banks -> GND
- J5 pad A57: 1V2_Banks -> GND
- J5 pad B03: 1V2_Banks -> GND
- J5 pad B04: 1V2_Banks -> GND
- J5 pad B07: 1V2_Banks -> GND
- J5 pad B08: 1V2_Banks -> GND
- J5 pad B11: 1V2_Banks -> GND
- J5 pad B14: 1V2_Banks -> GND
- J5 pad B17: 1V2_Banks -> GND
- J5 pad B20: 1V2_Banks -> GND
- J5 pad B23: 1V2_Banks -> GND
- J5 pad B26: 1V2_Banks -> GND
- J5 pad B29: 1V2_Banks -> GND
- J5 pad B32: 1V2_Banks -> GND
- J5 pad B35: 1V2_Banks -> GND
- J5 pad B38: 1V2_Banks -> GND
- J5 pad B41: 1V2_Banks -> GND
- J5 pad B42: 1V2_Banks -> 1V8_Banks
- J5 pad B43: 1V2_Banks -> GND
- J5 pad B47: 1V2_Banks -> GND
- J5 pad B51: 1V2_Banks -> GND
- J5 pad B55: 1V2_Banks -> GND
- J5 pad C01: 1V2_Banks -> GND
- J5 pad C02: 1V2_Banks -> GND
- J5 pad C05: 1V2_Banks -> GND
- J5 pad C06: 1V2_Banks -> GND
- J5 pad C09: 1V2_Banks -> GND
- J5 pad C10: 1V2_Banks -> GND
- J5 pad C13: 1V2_Banks -> GND
- J5 pad C16: 1V2_Banks -> GND
- J5 pad C19: 1V2_Banks -> GND
- J5 pad C22: 1V2_Banks -> GND
- J5 pad C25: 1V2_Banks -> GND
- J5 pad C28: 1V2_Banks -> GND
- J5 pad C31: 1V2_Banks -> GND
- J5 pad C34: 1V2_Banks -> GND
- J5 pad C37: 1V2_Banks -> GND
- J5 pad C40: 1V2_Banks -> GND
- J5 pad C43: 1V2_Banks -> GND
- J5 pad C44: 1V2_Banks -> 1V8_Banks
- J5 pad C45: 1V2_Banks -> GND
- J5 pad C49: 1V2_Banks -> GND
- J5 pad C53: 1V2_Banks -> GND
- J5 pad C57: 1V2_Banks -> GND
- J5 pad D03: 1V2_Banks -> GND
- J5 pad D04: 1V2_Banks -> GND
- J5 pad D07: 1V2_Banks -> GND
- J5 pad D08: 1V2_Banks -> GND
- J5 pad D11: 1V2_Banks -> GND
- J5 pad D14: 1V2_Banks -> GND
- J5 pad D17: 1V2_Banks -> GND
- J5 pad D20: 1V2_Banks -> GND
- J5 pad D23: 1V2_Banks -> GND
- J5 pad D26: 1V2_Banks -> GND
- J5 pad D29: 1V2_Banks -> GND
- J5 pad D32: 1V2_Banks -> GND
- J5 pad D35: 1V2_Banks -> GND
- J5 pad D38: 1V2_Banks -> GND
- J5 pad D41: 1V2_Banks -> GND
- J5 pad D42: 1V2_Banks -> 1V8_Banks
- J5 pad D43: 1V2_Banks -> GND
- J5 pad D47: 1V2_Banks -> GND
- J5 pad D51: 1V2_Banks -> GND
- J5 pad D55: 1V2_Banks -> GND
- J6 pad 10: 1V2_Banks -> GND
- J6 pad 6: 1V2_Banks -> GND
- LDO1 pad 3: 1V2_Banks -> GND
- LDO1 pad 6: 1V2_Banks -> GND
- LDO10 pad 3: 1V2_Banks -> GND
- LDO10 pad 6: 1V2_Banks -> GND
- LDO2 pad 3: 1V2_Banks -> GND
- LDO2 pad 6: 1V2_Banks -> GND
- LDO4 pad 3: 1V2_Banks -> GND
- LDO4 pad 6: 1V2_Banks -> GND
- LDO5 pad 3: 1V2_Banks -> GND
- LDO5 pad 6: 1V2_Banks -> GND
- LDO7 pad 3: 1V2_Banks -> GND
- LDO7 pad 6: 1V2_Banks -> GND
- LDO8 pad 3: 1V2_Banks -> GND
- LDO8 pad 6: 1V2_Banks -> GND
- LDO9 pad 3: 1V2_Banks -> GND
- LDO9 pad 6: 1V2_Banks -> GND
- Q4 pad 3: 1V2_Banks -> GND
- Q6 pad 3: 3V3_IO -> GND
- Q8 pad 3: 3V3_IO -> GND
- R11 pad 2: 1V2_Banks -> GND
- R14 pad 2: 1V2_Banks -> GND
- R22 pad 2: 3V3_IO -> GND
- R29 pad 1: 1V2_Banks -> GND
- R33 pad 2: 1V2_Banks -> GND
- R36 pad 2: 1V2_Banks -> GND
- R40 pad 2: 1V2_Banks -> GND
- R43 pad 2: 1V2_Banks -> GND
- R55 pad 2: 1V2_Banks -> GND
- R56 pad 2: 1V2_Banks -> GND
- R57 pad 2: 1V2_Banks -> GND
- R61 pad 2: 1V2_Banks -> GND
- R66 pad 2: 1V2_Banks -> GND
- R70 pad 1: 1V2_Banks -> GND
- R71 pad 1: 1V2_Banks -> GND
- R73 pad 1: 1V2_Banks -> GND
- R75 pad 1: 1V2_Banks -> GND
- R79 pad 1: 1V2_Banks -> GND
- R8 pad 1: 1V2_Banks -> GND
- R84 pad 1: 3V3_IO -> GND
- SW1 pad 1: 1V2_Banks -> GND
- SW1 pad 2: 1V2_Banks -> GND
- SW2 pad 1: 1V2_Banks -> GND
- SW2 pad 2: 1V2_Banks -> GND
- TP1 pad 1: 1V2_Banks -> GND
- TP13 pad 1: 1V2_Banks -> GND
- TP21 pad 1: 1V2_Banks -> GND
- TP23 pad 1: 1V2_Banks -> GND
- TP3 pad 1: 1V2_Banks -> GND
- TP5 pad 1: 1V2_Banks -> GND
- TP7 pad 1: 1V2_Banks -> GND
- TP9 pad 1: 1V2_Banks -> GND
- U1 pad 57: (no net) -> GND
- U10 pad 3: 1V2_Banks -> GND
- U10 pad 8: 1V2_Banks -> GND
- U11 pad 5: 1V2_Banks -> GND
- U11 pad 7: 1V2_Banks -> GND
- U12 pad 5: 1V2_Banks -> GND
- U12 pad 7: 1V2_Banks -> GND
- U16 pad 3: 1V2_Banks -> GND
- U2 pad 1: 1V2_Banks -> GND
- U3 pad 3: 1V2_Banks -> GND
- U3 pad 8: 1V2_Banks -> GND
- U4 pad 1: 1V2_Banks -> GND
- U5 pad 3: 1V2_Banks -> GND
- U6 pad C2: 1V2_Banks -> GND
- U6 pad C3: 1V2_Banks -> GND
- U7 pad 2: 1V2_Banks -> GND
- U7 pad 4: 1V2_Banks -> GND
- U7 pad 5: 1V2_Banks -> GND
- U7 pad 6: 1V2_Banks -> GND
- U8 pad 2: 1V2_Banks -> GND
- U8 pad 4: 1V2_Banks -> GND
- U8 pad 5: 1V2_Banks -> GND
- U8 pad 6: 1V2_Banks -> GND
- U9 pad 13: 1V2_Banks -> GND
- U9 pad 17: 1V2_Banks -> GND
- U9 pad 3: 1V2_Banks -> GND
- Y3 pad 2: 3V3_IO -> GND
Routing:
- net GND: track 0.00 -> 41.4 mm, vias 0 -> 65
- net /SOM240_1(1.5)/Peripherals_Ctrl1/READOUT8+: track 0.00 -> 14.4 mm
- net 1V8_Banks: track 0.00 -> 14.2 mm, vias 0 -> 4
- net VDD_BUCK_2V5: track 0.13 -> 14.2 mm, vias 0 -> 5
- net /SOM240_1(1.5)/Peripherals_Ctrl1/READOUT4+: track 0.00 -> 14.0 mm
- net /SOM240_1(1.5)/Peripherals_Ctrl1/READOUT5+: track 0.00 -> 11.8 mm
- net /SOM240_1(1.5)/Peripherals_Ctrl1/READOUT1+: track 0.00 -> 11.4 mm
- net /SOM240_1(1.5)/Peripherals_Ctrl1/READOUT6-: track 0.00 -> 11.4 mm
- net /SOM240_1(1.5)/Peripherals_Ctrl1/READOUT1-: track 0.00 -> 11.1 mm
- net /SOM240_1(1.5)/Peripherals_Ctrl1/READOUT5-: track 0.00 -> 11.1 mm
- net /SOM240_1(1.5)/Peripherals_Ctrl1/READOUT2-: track 0.00 -> 10.7 mm
- net /SOM240_1(1.5)/Peripherals_Ctrl1/READOUT8-: track 0.00 -> 10.2 mm
- net /SOM240_1(1.5)/Peripherals_Ctrl1/READOUT4-: track 0.00 -> 9.81 mm
- net /SOM240_1(1.5)/Peripherals_Ctrl1/READOUT7-: track 0.00 -> 8.37 mm
- net /SOM240_1(1.5)/Peripherals_Ctrl1/READOUT7+: track 0.00 -> 8.14 mm
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- added copper zone on In1.Cu, net GND
- added copper zone on In8.Cu, net GND
