File: PSEC5_Ctrl_Board/_autosave-PSEC5_Ctrl_Board.kicad_pcb (KiCad board)
At the start: 10 copper layers, 192.6 x 125.7 mm, 278 parts, among them J1 1766343, J10 ADM6-60-01.5-L-4-2-A-TR, J12 878311420, J14 ZX62D-B-5P830, J2 QSH-040-01-X-D-DP-A, J4 QSH-040-01-X-D-DP-A, J5 ADM6-60-01.5-L-4-2-A-TR (1), J6 1040310811, J9 1766343, Q4 NMOS, Q6 NMOS, Q8 NMOS, SW1 SW_MEC_5G, SW2 SW_MEC_5G, T1 7499111446, U1 88E1512-A0-NNP2C000, U10 PUSB3FR4Z, U11 TPS3808G01QDRVRQ1, U12 TPS3808G01QDRVRQ1, U14 SIA427ADJ-T1-GE3, U16 OKX-T/5-D12N-C, U2 LTC2600CGN_PBF, U3 PUSB3FR4Z, U4 LTC2600CGN_PBF, U5 OKX-T/5-D12N-C, U6 PI4ULS3V4857GEAEX, U7 MCP1501-25E/SN, U8 MCP1501-25E/SN, U9 FT230XQ-R, Y3 ASE2-25.000MHZ-ET

Commit message: again
Parts:
- C62, C64, L5: moved to B.Cu
- moved C62 82.7 mm to (77.2, 85.1), turned to 90 degrees
- moved C64 78.0 mm to (75.7, 85.1), turned to 90 degrees
- moved L5 74.0 mm to (74.2, 85.1), turned to -90 degrees
- moved C57 26.7 mm to (75.2, 72.1)
- moved R100 26.7 mm to (75.2, 73.7)
Routing:
- net /SOM240_1(1.5)/ADC_DOUT5-: track 20.0 -> 100.9 mm
- net /SOM240_1(1.5)/ADC_DOUT5+: track 20.9 -> 101.0 mm
- net Net-(T1-SHIELD1): track 1.47 -> 15.9 mm
- net GND: track 281.4 -> 287.2 mm, vias 243 -> 245
- net /SOM240_1(1.5)/ethernet1/PHY_VCC: track 6.42 -> 11.2 mm
- net 3V3_IO: track 42.3 -> 46.6 mm, vias 13 -> 14
- net /SOM240_1(1.5)/SDI_DAC_THRES: track 24.0 -> 25.6 mm
- net /SOM240_1(1.5)/SDI_DAC_BIAS: track 113.7 -> 115.2 mm
- net /SOM240_1(1.5)/ethernet1/PHY_MDI0_P: vias 0 -> 1
- net /SOM240_1(1.5)/ethernet1/PHY_MDI0_N: vias 0 -> 1

Commit message: more changes, adc net names driving me crazy
Parts:
- removed J9: 1766343, Connector_Phoenix_GMSTB:PhoenixContact_GMSTBA_2,5_2-G_1x02_P7.50mm_Horizontal
- C116, C117, C33, C34, C35, C36, C37, C38, C39, C40, C73, C75, C78, C79, R56, R57: moved to B.Cu
- moved C44 162.0 mm to (90.2, 89.7)
- moved C42 157.1 mm to (86.6, 99.1)
- moved R65 157.1 mm to (91.8, 99.1)
- moved U11 151.3 mm to (85.9, 88.9)
- moved C45 150.3 mm to (81.3, 89.7), turned to 180 degrees
- moved R20 65.4 mm to (223.3, 82.5), turned to 180 degrees
- moved R21 62.4 mm to (223.3, 81.0), turned to 180 degrees
- moved R57 62.2 mm to (237.5, 79.8), turned to -90 degrees
- moved R56 62.2 mm to (217.4, 79.2), turned to -90 degrees
- moved C73 60.3 mm to (238.0, 75.7)
- moved C33 57.4 mm to (234.2, 71.9), turned to 90 degrees
- moved C37 57.2 mm to (213.6, 71.6), turned to 90 degrees
- moved C78 56.5 mm to (217.4, 75.7)
- moved C75 55.7 mm to (238.0, 74.2)
- moved C38 55.7 mm to (215.1, 71.6), turned to 90 degrees
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Connections:
- J1 pad 2: unconnected-(J1-Pad2) -> Net-(U16-+VIN)
Routing:
- net GND: track 287.2 -> 339.8 mm, vias 245 -> 273
- net 1V8_ADC: track 0.00 -> 48.1 mm, vias 0 -> 16
- net 1V8_Banks: track 23.0 -> 3.30 mm, vias 8 -> 2
- net Net-(U16-+VIN): track 12.3 -> 0.00 mm
- net Net-(U5-+VIN): track 10.4 -> 0.00 mm
- net Net-(ADC2-REFT): track 0.00 -> 7.63 mm, vias 0 -> 1
- net Net-(ADC1-VREF): track 0.00 -> 6.84 mm, vias 0 -> 1
- net Net-(ADC1-REFT): track 0.00 -> 5.50 mm, vias 0 -> 1
- net Net-(ADC2-REFB): track 0.00 -> 5.33 mm, vias 0 -> 1
- net Net-(ADC1-REFB): track 0.00 -> 5.00 mm, vias 0 -> 1
- net Net-(ADC2-VREF): track 0.00 -> 4.78 mm, vias 0 -> 1
- net Net-(ADC1-RBIAS): track 0.00 -> 3.33 mm, vias 0 -> 1
- net Net-(ADC2-RBIAS): track 0.00 -> 3.06 mm, vias 0 -> 1
- net /SOM240_1(1.5)/ADC2_SCLK/DTP: track 0.06 -> 3.08 mm
- net /SOM240_1(1.5)/ADC2_SDIO/ODM: track 0.15 -> 3.14 mm
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