File: PSEC5_Ctrl_Board/ethernet.kicad_sch (KiCad schematic)
At the start: 42 parts, among them Q6 NMOS, Q8 NMOS, T1 7499111446, U1 88E1512-A0-NNP2C000, Y3 ASE2-25.000MHZ-ET

Commit message: Round 1 changes done
Connections:
- net GND: now also U1.12 (LED[2]/INTn)
- net LED_11: now also U1.13 (LED[1])
- net LED_12: no longer U1.12 (LED[2]/INTn)
- net LED_13: now also U1.14 (LED[0]); no longer U1.13 (LED[1])
- net LED_14: no longer U1.14 (LED[0])
Changed lines of the file:
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@@
 	(wire
 		(pts
+			(xy 90.17 109.22) (xy 90.17 107.95)
+		)
+		(stroke
+			(width 0)
+			(type default)
+		)
+	)
+	(wire
+		(pts
 			(xy 39.37 154.94) (xy 39.37 157.48)
 		)
@@
 	(wire
 		(pts
-			(xy 96.52 105.41) (xy 106.68 105.41)
+			(xy 90.17 107.95) (xy 106.68 107.95)
 		)
 		(stroke
@@
 	(wire
 		(pts
-			(xy 96.52 107.95) (xy 106.68 107.95)
-		)
-		(stroke
-			(width 0)
-			(type default)
-		)
-	)
-	(wire
-		(pts
 			(xy 96.52 128.27) (xy 106.68 128.27)
 		)
@@
 	(wire
 		(pts
+			(xy 90.17 105.41) (xy 106.68 105.41)
+		)
+		(stroke
+			(width 0)
+			(type default)
+		)
+	)
+	(wire
+		(pts
 			(xy 232.41 19.05) (xy 242.57 19.05)
 		)
@@
 		)
 	)
-	(label "LED_12"
-		(at 96.52 107.95 0)
-		(fields_autoplaced yes)
-		(effects
-			(font
-				(size 1.27 1.27)
-			)
-			(justify left bottom)
-		)
-	)
 	(label "PHY_MDI2_P"
 		(at 96.52 130.81 180)
@@
 	)
 	(label "VDDO"
-		(at 96.52 105.41 180)
+		(at 90.17 105.41 180)
 		(fields_autoplaced yes)
 		(effects
@@
 		)
 	)
-	(label "LED_13"
+	(label "LED_11"
 		(at 96.52 110.49 0)
 		(fields_autoplaced yes)
@@
 		)
 	)
-	(label "LED_14"
+	(label "LED_13"
 		(at 96.52 113.03 0)
 		(fields_autoplaced yes)
@@
 					(unit 1)
 				)
+			)
+		)
+	)
+	(symbol
+		(lib_id "power:GND")
+		(at 90.17 109.22 0)
+		(unit 1)
+		(exclude_from_sim no)
+		(in_bom yes)
+		(on_board yes)
+		(dnp no)
+		(property "Reference" "#PWR067"
+			(at 90.17 115.57 0)
+			(effects
+				(font
+					(size 1.27 1.27)
+				)
+				(hide yes)
+			)
+		)
+		(property "Value" "GND"
+			(at 86.614 110.236 0)
+			(effects
+				(font
+					(size 1.27 1.27)
+				)
+			)
+		)
+		(property "Footprint" ""
+			(at 90.17 109.22 0)
+			(effects
+				(font
+					(size 1.27 1.27)
+				)
+				(hide yes)
+			)
+		)
+		(property "Datasheet" ""
+			(at 90.17 109.22 0)
+			(effects
+				(font
+					(size 1.27 1.27)
+				)
+				(hide yes)
+			)
+		)
+		(property "Description" "Power symbol creates a global label with name \"GND\" , ground"
+			(at 90.17 109.22 0)
+			(effects
+				(font
+					(size 1.27 1.27)
+				)
+				(hide yes)
+			)
+		)
+		(pin "1"
+		)
+		(instances
+			(project ""
+				(path "/165f2ae6-d522-4adf-a6c4-bb137b209d33/1f6d7a03-cfad-4370-8d2b-49ab19e248d8/6e9ff0d5-3c45-486c-9945-94fa6223df4a"
+					(reference "#PWR067")
+					(unit 1)
+				)

Commit message: V2
Parts:
- added R112, R113: 10k, Resistor_SMD:R_0603_1608Metric, symbol Device:R_Small_US
- added R114, R115: 0R, Resistor_SMD:R_0603_1608Metric, symbol Device:R_Small_US
Connections:
- net GND: no longer U1.12 (LED[2]/INTn)
- net LED_11: no longer names the net of R74.1, T1.11
- net LED_11: no longer Q8.1 (D), U1.13 (LED[1])
- net LED_12: no longer names the net of T1.12
- net LED_12: now also R114.1; no longer Q8.2 (G)
- net LED_13: no longer names the net of R76.1, T1.13
- net LED_13: no longer Q6.1 (D), U1.14 (LED[0])
- net LED_14: no longer names the net of Q6.2 (G)
- net LED_14: now also R113.2; no longer T1.14
- new net: Q6.1 (D), R115.2
- new net: R115.1, T1.14
- new net: Q8.1 (D), R114.2
- new net: Q8.2 (G), R112.2
- new net ETH_LED0: R112.1, U1.14 (LED[0])
- new net ETH_LED1: R113.1, U1.13 (LED[1])
- no-connect marks 9 -> 10
Other:
- moved on the sheet: Q6, Q8, R74, R76
