File: PSEC5_Ctrl_Board/Translator_Board/To Ctrl.kicad_sch (KiCad schematic)
At the start: 2 parts, among them J1 QTH-040-01-X-D-DP-A, J9 QTH-040-01-X-D-DP-A

Commit message: Translator Schematic, Initial Touches to Layout
Parts:
- added H10, H11, H12, H9: MountingHole, MountingHole:MountingHole_2.7mm, symbol Mechanical:MountingHole

Commit message: Translator Board push
Parts:
- removed H10, H11, H12, H9: MountingHole, MountingHole:MountingHole_2.7mm, symbol Mechanical:MountingHole
Connections:
- net DISCBIAS: now also J1.09; no longer J1.49
- net Disc_Thresh1: now also J1.21; no longer J1.61
- net Disc_Thresh2: now also J1.25; no longer J1.65
- net Disc_Thresh3: now also J1.29; no longer J1.69
- net Disc_Thresh4: now also J1.33; no longer J1.73
- net Disc_Thresh5: now also J1.37; no longer J1.77
- net Disc_Thresh6: now also J1.69; no longer J1.29
- net Disc_Thresh7: now also J1.73; no longer J1.33
- net Disc_Thresh8: now also J1.77; no longer J1.37
- net P5_ReadClk: now also J1.52; no longer J1.12
- net P5_rst: now also J1.20; no longer J1.60
- net PICO: now also J1.28; no longer J1.68
- net POCI: now also J1.26; no longer J1.66
- net Psec5RefClk: now also J1.35; no longer J1.75
- net Psec5TriggerIn: now also J1.78; no longer J1.38
- net Psec5TriggerOut: now also J1.50; no longer J1.10
- net READBIAS1: now also J1.07; no longer J1.47
- net READBIAS2: now also J1.05; no longer J1.45
- net SIGNAL1+: now also J1.06; no longer J1.46
- net SIGNAL1-: now also J1.08; no longer J1.48
- net SIGNAL2+: now also J1.14; no longer J1.54
- net SIGNAL2-: now also J1.16; no longer J1.56
- net SIGNAL3+: now also J1.22; no longer J1.62
- net SIGNAL3-: now also J1.24; no longer J1.64
- net SIGNAL4+: now also J1.30; no longer J1.70
- net SIGNAL4-: now also J1.32; no longer J1.72
- net SIGNAL5+: now also J1.46; no longer J1.06
- net SIGNAL5-: now also J1.48; no longer J1.08
- net SIGNAL6+: now also J1.54; no longer J1.14
- net SIGNAL6-: now also J1.56; no longer J1.16
- net SIGNAL7+: now also J1.62; no longer J1.22
- net SIGNAL7-: now also J1.64; no longer J1.24
- net SIGNAL8+: now also J1.70; no longer J1.30
- net SIGNAL8-: now also J1.72; no longer J1.32
- net SPIclk: now also J1.18; no longer J1.58
- net V_ped1: no longer J9.38
- net WBUFBIAS: now also J1.11; no longer J1.51
- new net V_ped2: J9.38
