File: PSEC5_Ctrl_Board/Translator_Board/To DUT.kicad_sch (KiCad schematic)
At the start: 6 parts, among them J4 QSH-040-01-X-D-DP-A, J5 QSH-040-01-X-D-DP-A

Commit message: Translator Schematic, Initial Touches to Layout
Parts:
- removed H4: MountingHole, MountingHole:MountingHole_2.2mm_M2, symbol Mechanical:MountingHole
- added H8: MountingHole, MountingHole:MountingHole_2.7mm, symbol Mechanical:MountingHole
- H5, H6, H7: footprint MountingHole:MountingHole_2.2mm_M2 -> MountingHole:MountingHole_2.7mm
Changed lines of the file:
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@@
+	)
+	(symbol
+		(lib_id "Mechanical:MountingHole")
+		(at 120.65 137.16 0)
+		(unit 1)
+		(exclude_from_sim yes)
+		(in_bom no)
+		(on_board yes)
+		(dnp no)
+		(fields_autoplaced yes)
+		(property "Reference" "H6"
+			(at 123.19 135.8899 0)
+			(effects
+				(font
+					(size 1.27 1.27)
+				)
+				(justify left)
+			)
+		)
+		(property "Value" "MountingHole"
+			(at 123.19 138.4299 0)
+			(effects
+				(font
+					(size 1.27 1.27)
+				)
+				(justify left)
+			)
+		)
+		(property "Footprint" "MountingHole:MountingHole_2.7mm"
+			(at 120.65 137.16 0)
+			(effects
+				(font
+					(size 1.27 1.27)
+				)
+				(hide yes)
+			)
+		)
+		(property "Datasheet" "~"
+			(at 120.65 137.16 0)
+			(effects
+				(font
+					(size 1.27 1.27)
+				)
+				(hide yes)
+			)
+		)
+		(property "Description" "Mounting Hole without connection"
+			(at 120.65 137.16 0)
+			(effects
+				(font
+					(size 1.27 1.27)
+				)
+				(hide yes)
+			)
+		)
+		(instances
+			(project "Translator_Board"
+				(path "/03aee455-6aac-4c5b-b9dc-8dd41334d4bb/4f60dabf-a622-4c11-808c-a83228c2f00b"
+					(reference "H6")
+					(unit 1)
+				)
+			)
+		)
 	)
 	(symbol
@@
 	(symbol
 		(lib_id "Mechanical:MountingHole")
-		(at 256.54 137.16 0)
+		(at 260.35 137.16 0)
 		(unit 1)
 		(exclude_from_sim yes)
@@
 		(dnp no)
 		(fields_autoplaced yes)
-		(property "Reference" "H4"
-			(at 259.08 135.8899 0)
+		(property "Reference" "H8"
+			(at 262.89 135.8899 0)
 			(effects
 				(font
@@
 		)
 		(property "Value" "MountingHole"
-			(at 259.08 138.4299 0)
+			(at 262.89 138.4299 0)
 			(effects
 				(font
@@
 			)
 		)
-		(property "Footprint" "MountingHole:MountingHole_2.2mm_M2"
-			(at 256.54 137.16 0)
+		(property "Footprint" "MountingHole:MountingHole_2.7mm"
+			(at 260.35 137.16 0)
 			(effects
 				(font
@@
 		)
 		(property "Datasheet" "~"
-			(at 256.54 137.16 0)
+			(at 260.35 137.16 0)
 			(effects
 				(font
@@
 		)
 		(property "Description" "Mounting Hole without connection"
-			(at 256.54 137.16 0)
+			(at 260.35 137.16 0)
 			(effects
 				(font
@@
 			(project "Translator_Board"
 				(path "/03aee455-6aac-4c5b-b9dc-8dd41334d4bb/4f60dabf-a622-4c11-808c-a83228c2f00b"
-					(reference "H4")
+					(reference "H8")
+					(unit 1)
+				)
+			)
+		)
+	)
+	(symbol
+		(lib_id "Mechanical:MountingHole")
+		(at 201.93 138.43 0)
+		(unit 1)
+		(exclude_from_sim yes)
+		(in_bom no)
+		(on_board yes)
+		(dnp no)
+		(fields_autoplaced yes)
+		(property "Reference" "H7"
+			(at 204.47 137.1599 0)
+			(effects
+				(font
+					(size 1.27 1.27)
+				)
+				(justify left)
+			)
+		)
+		(property "Value" "MountingHole"
+			(at 204.47 139.6999 0)
+			(effects
+				(font
+					(size 1.27 1.27)
+				)
+				(justify left)
+			)
+		)
+		(property "Footprint" "MountingHole:MountingHole_2.7mm"
+			(at 201.93 138.43 0)
+			(effects
+				(font
+					(size 1.27 1.27)
+				)
+				(hide yes)
+			)
+		)
+		(property "Datasheet" "~"
+			(at 201.93 138.43 0)
+			(effects
+				(font
+					(size 1.27 1.27)
+				)
+				(hide yes)
+			)
+		)
+		(property "Description" "Mounting Hole without connection"
+			(at 201.93 138.43 0)
+			(effects
+				(font
+					(size 1.27 1.27)
+				)
+				(hide yes)
+			)
+		)
+		(instances
+			(project "Translator_Board"
+				(path "/03aee455-6aac-4c5b-b9dc-8dd41334d4bb/4f60dabf-a622-4c11-808c-a83228c2f00b"
+					(reference "H7")
 					(unit 1)
 				)
@@
 	)
 	(symbol
-		(lib_id "Mechanical:MountingHole")
-		(at 123.19 137.16 0)
-		(unit 1)
-		(exclude_from_sim yes)
-		(in_bom no)
-		(on_board yes)
-		(dnp no)
-		(fields_autoplaced yes)
-		(property "Reference" "H6"
-			(at 125.73 135.8899 0)
-			(effects
-				(font
-					(size 1.27 1.27)
-				)
-				(justify left)
-			)
-		)
-		(property "Value" "MountingHole"
-			(at 125.73 138.4299 0)
-			(effects
-				(font
-					(size 1.27 1.27)
-				)
-				(justify left)
-			)
-		)
-		(property "Footprint" "MountingHole:MountingHole_2.2mm_M2"
-			(at 123.19 137.16 0)
-			(effects
-				(font
-					(size 1.27 1.27)
-				)
-				(hide yes)
-			)
-		)
-		(property "Datasheet" "~"
-			(at 123.19 137.16 0)
-			(effects
-				(font
-					(size 1.27 1.27)
-				)
-				(hide yes)
-			)
-		)
-		(property "Description" "Mounting Hole without connection"
-			(at 123.19 137.16 0)
-			(effects
-				(font
-					(size 1.27 1.27)
-				)
-				(hide yes)
-			)
-		)
-		(instances
-			(project "Translator_Board"
-				(path "/03aee455-6aac-4c5b-b9dc-8dd41334d4bb/4f60dabf-a622-4c11-808c-a83228c2f00b"
-					(reference "H6")
-					(unit 1)
-				)
-			)
-		)
-	)
-	(symbol
 		(lib_id "QSH-040-01-X-D-DP-A:QSH-040-01-X-D-DP-A")
 		(at 48.26 74.93 0)
@@
 			)
 		)
-		(property "Footprint" "MountingHole:MountingHole_2.2mm_M2"
+		(property "Footprint" "MountingHole:MountingHole_2.7mm"
 			(at 49.53 135.89 0)
 			(effects
@@
 					(unit 1)
 				)
-			)
-		)
-	)
-	(symbol
-		(lib_id "Mechanical:MountingHole")
-		(at 200.66 135.89 0)
-		(unit 1)
-		(exclude_from_sim yes)
-		(in_bom no)
-		(on_board yes)
-		(dnp no)
-		(fields_autoplaced yes)
-		(property "Reference" "H7"
-			(at 203.2 134.6199 0)
-			(effects
-				(font
-					(size 1.27 1.27)
-				)
-				(justify left)
-			)
-		)
-		(property "Value" "MountingHole"
-			(at 203.2 137.1599 0)
-			(effects
-				(font
-					(size 1.27 1.27)
-				)
-				(justify left)
-			)
-		)
-		(property "Footprint" "MountingHole:MountingHole_2.2mm_M2"
-			(at 200.66 135.89 0)
-			(effects
-				(font
-					(size 1.27 1.27)
-				)
-				(hide yes)
-			)
-		)
-		(property "Datasheet" "~"
-			(at 200.66 135.89 0)
-			(effects
-				(font
-					(size 1.27 1.27)
-				)
-				(hide yes)
-			)
-		)
-		(property "Description" "Mounting Hole without connection"
-			(at 200.66 135.89 0)
-			(effects
-				(font
-					(size 1.27 1.27)
-				)
-				(hide yes)
-			)
-		)
-		(instances
-			(project "Translator_Board"
-				(path "/03aee455-6aac-4c5b-b9dc-8dd41334d4bb/4f60dabf-a622-4c11-808c-a83228c2f00b"
-					(reference "H7")
-					(unit 1)
-				)

Commit message: Translator Board push
Parts:
- H5, H6, H7, H8: footprint MountingHole:MountingHole_2.7mm -> MountingHole:MountingHole_2.1mm
