File: PSEC5_Ctrl_Board/Translator_Board/Translator_Board.kicad_pcb (KiCad board)
At the start: 2 copper layers, 75 x 110 mm, 16 parts, among them J1 QTH-040-01-X-D-DP-A, J4 QSH-040-01-X-D-DP-A, J5 QSH-040-01-X-D-DP-A, J9 QTH-040-01-X-D-DP-A

Commit message: Translator Board push
Parts:
- removed H10, H11, H12, H9: MountingHole, MountingHole:MountingHole_2.7mm
- H5, H6, H7, H8: footprint MountingHole:MountingHole_2.7mm -> MountingHole:MountingHole_2.1mm
- J1, J9: moved to B.Cu
- moved H6 115.6 mm to (123.8, 46.5)
- moved TP1 115.1 mm to (116.0, 79.5)
- moved TP2 115.1 mm to (116.0, 84.5)
- moved TP3 115.1 mm to (116.0, 89.6)
- moved TP4 115.1 mm to (116.0, 94.7)
- moved H5 101.3 mm to (169.4, 46.5)
- moved H7 94.7 mm to (123.8, 117.4)
- moved H8 50.0 mm to (169.4, 117.4)
- moved J1 14.5 mm to (146.6, 49.0), turned to 180 degrees
- moved J9 13.0 mm to (146.6, 115.1), turned to 180 degrees
- turned J4 to 180 degrees
Connections:
- J1 pad 05: unconnected-(J1-Pad05) -> READBIAS2
- J1 pad 06: ADC5_Out+ -> ADC1_Out+
- J1 pad 07: unconnected-(J1-Pad07) -> READBIAS1
- J1 pad 08: ADC5_Out- -> ADC1_Out-
- J1 pad 09: unconnected-(J1-Pad09) -> DISCBIAS
- J1 pad 10: Psec5TriggerOut -> unconnected-(J1-Pad10)
- J1 pad 11: unconnected-(J1-Pad11) -> WBUFBIAS
- J1 pad 12: P5_ReadClk -> unconnected-(J1-Pad12)
- J1 pad 14: ADC6_Out+ -> ADC2_Out+
- J1 pad 16: ADC6_Out- -> ADC2_Out-
- J1 pad 18: unconnected-(J1-Pad18) -> SPIclk
- J1 pad 20: unconnected-(J1-Pad20) -> P5_rst
- J1 pad 21: unconnected-(J1-Pad21) -> Disc_Thresh1
- J1 pad 22: ADC7_Out+ -> ADC3_Out+
- J1 pad 24: ADC7_Out- -> ADC3_Out-
- J1 pad 25: unconnected-(J1-Pad25) -> Disc_Thresh2
- J1 pad 26: unconnected-(J1-Pad26) -> POCI
- J1 pad 28: unconnected-(J1-Pad28) -> PICO
- J1 pad 29: Disc_Thresh6 -> Disc_Thresh3
- J1 pad 30: ADC8_Out+ -> ADC4_Out+
- J1 pad 32: ADC8_Out- -> ADC4_Out-
- J1 pad 33: Disc_Thresh7 -> Disc_Thresh4
- J1 pad 35: unconnected-(J1-Pad35) -> PSEC5_CLK_OUT
- J1 pad 37: Disc_Thresh8 -> Disc_Thresh5
- J1 pad 38: Psec5TriggerIn -> unconnected-(J1-Pad38)
- J1 pad 45: READBIAS2 -> unconnected-(J1-Pad45)
- J1 pad 46: ADC1_Out+ -> ADC5_Out+
- J1 pad 47: READBIAS1 -> unconnected-(J1-Pad47)
- J1 pad 48: ADC1_Out- -> ADC5_Out-
- J1 pad 49: DISCBIAS -> unconnected-(J1-Pad49)
- J1 pad 50: unconnected-(J1-Pad50) -> Psec5TriggerOut
- J1 pad 51: WBUFBIAS -> unconnected-(J1-Pad51)
- J1 pad 52: unconnected-(J1-Pad52) -> P5_ReadClk
- J1 pad 54: ADC2_Out+ -> ADC6_Out+
- J1 pad 56: ADC2_Out- -> ADC6_Out-
- J1 pad 58: SPIclk -> unconnected-(J1-Pad58)
- J1 pad 60: P5_rst -> unconnected-(J1-Pad60)
- J1 pad 61: Disc_Thresh1 -> unconnected-(J1-Pad61)
- J1 pad 62: ADC3_Out+ -> ADC7_Out+
- J1 pad 64: ADC3_Out- -> ADC7_Out-
- J1 pad 65: Disc_Thresh2 -> unconnected-(J1-Pad65)
- J1 pad 66: POCI -> unconnected-(J1-Pad66)
- J1 pad 68: PICO -> unconnected-(J1-Pad68)
- J1 pad 69: Disc_Thresh3 -> Disc_Thresh6
- J1 pad 70: ADC4_Out+ -> ADC8_Out+
- J1 pad 72: ADC4_Out- -> ADC8_Out-
- J1 pad 73: Disc_Thresh4 -> Disc_Thresh7
- J1 pad 75: PSEC5_CLK_OUT -> unconnected-(J1-Pad75)
- J1 pad 77: Disc_Thresh5 -> Disc_Thresh8
- J1 pad 78: unconnected-(J1-Pad78) -> Psec5TriggerIn
- J4 pad 50: TRIGGEROUT -> Psec5TriggerOut
- J4 pad 52: ReadClk -> P5_ReadClk
- J5 pad 43: V_ped1 -> V_ped2
- J9 pad 01: HPB01_P -> GND
- J9 pad 03: HPB01_N -> GND
- J9 pad 05: HPB00_CC_P -> GND
- J9 pad 07: HPB00_CC_N -> GND
- J9 pad 09: HPB_CLK0_P -> GND
- J9 pad 11: HPB_CLK0_N -> GND
- J9 pad 13: HPB04_P -> GND
- J9 pad 15: HPB04_N -> GND
- J9 pad 17: HPB17_P -> GND
- J9 pad 19: HPB17_N -> GND
- J9 pad 21: HPC09_P -> GND
- J9 pad 23: HPC09_N -> GND
- J9 pad 25: HPC01_P -> GND
- J9 pad 27: HPC01_N -> GND
- J9 pad 29: HPC00_CC_P -> GND
- J9 pad 31: HPC00_CC_N -> GND
- J9 pad 33: HPC02_P -> GND
- J9 pad 35: HPC02_N -> GND
- J9 pad 37: HPC04_P -> GND
- J9 pad 38: V_ped1 -> V_ped2
- J9 pad 39: HPC04_N -> GND
- J9 pad 58: ADC_SCLK -> ADC_SCK
Routing:
- net ADC3_Out+: track 0.00 -> 8.39 mm, vias 0 -> 1
- net Disc_Thresh5: track 0.00 -> 7.73 mm, vias 0 -> 1
- net SPIclk: track 0.00 -> 7.39 mm, vias 0 -> 1
- net ADC7_Out+: track 0.00 -> 7.39 mm, vias 0 -> 1
- net ADC6_Out+: track 0.00 -> 7.39 mm, vias 0 -> 1
- net ADC3_Out-: track 0.00 -> 7.31 mm, vias 0 -> 1
- net PSEC5_CLK_OUT: track 0.00 -> 7.26 mm, vias 0 -> 1
- net ADC5_Out-: track 0.00 -> 7.17 mm, vias 0 -> 1
- net Psec5TriggerOut: track 0.00 -> 6.39 mm, vias 0 -> 1
- net ADC8_Out+: track 0.00 -> 6.39 mm, vias 0 -> 1
- net ADC4_Out+: track 0.00 -> 6.39 mm, vias 0 -> 1
- net POCI: track 0.00 -> 6.39 mm, vias 0 -> 1
- net Disc_Thresh8: track 0.00 -> 6.32 mm, vias 0 -> 1
- net DISCBIAS: track 0.00 -> 6.32 mm, vias 0 -> 1
- net P5_rst: track 0.00 -> 6.31 mm, vias 0 -> 1
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
Commit message: Translator Board Layout (Except power), DUT copy in main branch
DUT copy is under DUT_copy(1)
Parts:
- turned J5 to 180 degrees
Routing:
- net V_ped8: track 0.00 -> 92.9 mm, vias 0 -> 3
- net V_ped7: track 0.00 -> 89.6 mm, vias 0 -> 3
- net SYNC_N: track 0.00 -> 89.0 mm, vias 0 -> 3
- net V_ped6: track 0.00 -> 86.2 mm, vias 0 -> 3
- net DAC_SCLK: track 0.00 -> 82.7 mm, vias 0 -> 3
- net V_ped5: track 0.00 -> 80.7 mm, vias 0 -> 3
- net ADC_SDI: track 0.00 -> 78.2 mm, vias 0 -> 3
- net V_ped4: track 0.00 -> 76.5 mm, vias 0 -> 3
- net ADC_SCK: track 0.00 -> 74.6 mm, vias 0 -> 3
- net V_ped3: track 0.00 -> 71.1 mm, vias 0 -> 3
- net ADC_SDO: track 0.00 -> 69.6 mm, vias 0 -> 3
- net V_ped2: track 0.00 -> 66.2 mm, vias 0 -> 3
- net ADC_CNV: track 0.00 -> 65.3 mm, vias 0 -> 3
- net V_ped1: track 0.00 -> 61.7 mm, vias 0 -> 3
- net DAC_V_IN: track 0.00 -> 60.7 mm, vias 0 -> 3
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Other:
- copper layers 2 -> 4

Commit message: Translator Board v1
Parts:
- added TP5: ChipClk, TestPoint:TestPoint_THTPad_3.0x3.0mm_Drill1.5mm, F.Cu at (146.6, 37.5)
- moved TP2 19.2 mm to (113.0, 103.5)
- moved TP4 16.1 mm to (113.0, 110.5)
- moved TP1 11.4 mm to (113.0, 90.5)
- moved TP3 7.98 mm to (113.0, 97.0)
Connections:
- J5 pad 69: GND -> VDD50
- J5 pad 71: GND -> VDD50
- J9 pad 01: GND -> HPB01_P
- J9 pad 03: GND -> HPB01_N
- J9 pad 05: GND -> HPB00_CC_P
- J9 pad 07: GND -> HPB00_CC_N
- J9 pad 09: GND -> HPB_CLK0_P
- J9 pad 11: GND -> HPB_CLK0_N
- J9 pad 13: GND -> HPB04_P
- J9 pad 15: GND -> HPB04_N
- J9 pad 17: GND -> HPB17_P
- J9 pad 19: GND -> HPB17_N
- J9 pad 21: GND -> HPC09_P
- J9 pad 23: GND -> HPC09_N
- J9 pad 25: GND -> HPC01_P
- J9 pad 27: GND -> HPC01_N
- J9 pad 29: GND -> HPC00_CC_P
- J9 pad 31: GND -> HPC00_CC_N
- J9 pad 33: GND -> HPC02_P
- J9 pad 35: GND -> HPC02_N
- J9 pad 37: GND -> HPC04_P
- J9 pad 39: GND -> HPC04_N
- J9 pad 41: GND -> HPC15_CC_N
- J9 pad 43: GND -> HPC15_CC_P
- J9 pad 45: GND -> HPC14_N
- J9 pad 47: GND -> HPC14_P
- J9 pad 49: GND -> HPC19_N
- J9 pad 51: GND -> HPC19_P
- J9 pad 53: GND -> HPC08_N
- J9 pad 55: GND -> HPC08_P
- J9 pad 57: GND -> HPB19_N
- J9 pad 59: GND -> HPB19_P
- J9 pad 61: GND -> HPB16_N
- J9 pad 63: GND -> HPB16_P
- J9 pad 65: GND -> HPB06_N
- J9 pad 67: GND -> HPB06_P
- J9 pad 69: GND -> HPB12_N
- J9 pad 71: GND -> HPB12_P
- J9 pad 73: GND -> HPB08_N
- J9 pad 75: GND -> HPB08_P
- J9 pad 77: GND -> HPB15_CC_N
- J9 pad 79: GND -> HPB15_CC_P
Routing:
- net GND: track 38.0 -> 3.73 mm
- net 2V5_DUT: track 5.93 -> 38.2 mm
- net 1V8_DUT: track 5.83 -> 32.8 mm
- net 3V3_DUT: track 5.56 -> 26.7 mm
- net PSEC5_CLK_OUT: track 7.26 -> 14.2 mm
- net 1V2_DUT: track 3.70 -> 5.20 mm
- net VDD50: track 0.00 -> 0.50 mm
- added copper zone on In1.Cu, net 1V2_DUT
- added copper zone on In1.Cu, net 1V8_DUT
- added copper zone on In2.Cu, net 2V5_DUT
- added copper zone on In2.Cu, net 3V3_DUT
- added copper zone on B.Cu, net GND
- added copper zone on F.Cu, net GND
