File: KADC_CONTROLLER/_autosave-power_1.kicad_sch (KiCad schematic)
At the start: 3 parts, among them U1 OKX-T/5-D12N-C, U3 AP2127K-ADJTRG1

Commit message: Building out New Schematic
Finished KADC Power rails, creating new Kria K26 Symbol with correct net names, SOM1 DONE. SOM2, AB DONE, CD left to do
Parts:
- removed 1: LP38501TS-ADJ/NOPB, TS5B, symbol ul_LP38501TS-ADJ-NOPB:LP38501TS-ADJ_NOPB
- removed U3: AP2127K-ADJTRG1, AP2127K-ADJTRG1_DIO, symbol AP2127K_ADJTRG1:AP2127K-ADJTRG1
- added C1, C10, C2, C22, C6, C7, C8, C9: 10u, Capacitor_SMD:C_0603_1608Metric, symbol Device:C_Small
- added C3: 1u, symbol Device:C_Small
- added C4: 0.1u, symbol Device:C_Small
- added C5: 10u, symbol Device:C_Small
- added J1: 1766343, CONN_1766343_PXC, symbol 1766343:1766343
- added LDO1, LDO2, LDO3, LDO4: LP38501TS-ADJ/NOPB, ul_LP38501TS-ADJ-NOPB:TS5B, symbol PSEC5_ctrlbd:LP38501TS-ADJ_NOPB
- added R1: 1.47k, symbol Device:R_Small_US
- added R10: 11.3k, Resistor_SMD:R_0603_1608Metric, symbol Device:R_Small_US
- added R11, R12, R15, R3, R59, R61, R7, R8: 10k, Resistor_SMD:R_0603_1608Metric, symbol Device:R_Small_US
- added R13: 34k, Resistor_SMD:R_0603_1608Metric, symbol Device:R_Small_US
- added R14: 10.5k, Resistor_SMD:R_0603_1608Metric, symbol Device:R_Small_US
- added R16: 0R, symbol Device:R_Small_US
- added R17: FIXED, symbol Device:R_Small_US
- added R2: 4.42k, symbol Device:R_Small_US
- added R4, R60: 14.7k, Resistor_SMD:R_0603_1608Metric, symbol Device:R_Small_US
- added R5, R82: 4.99k, Resistor_SMD:R_0603_1608Metric, symbol Device:R_Small_US
- added R6: 10k, symbol Device:R_Small_US
- added R9: 20k, Resistor_SMD:R_0603_1608Metric, symbol Device:R_Small_US
- added TP1, TP14, TP3, TP5: 1V8_Bank, TestPoint:TestPoint_THTPad_1.5x1.5mm_Drill0.7mm, symbol Connector:TestPoint
- added TP13, TP2, TP4, TP6: GND, TestPoint:TestPoint_THTPad_1.5x1.5mm_Drill0.7mm, symbol Connector:TestPoint
- added U2: AD5274BCPZ-100-RL7, CP_10_9_ADI, symbol AD5274BCPZ_100_RL7:AD5274BCPZ-100-RL7
- added U4, U5: OKX-T/5-D12N-C, OKX-T/5-D12N-C_MUR, symbol OKX_T_5_D12N_C:OKX-T_5-D12N-C
Connections:
- net VDD_BUCK_5V: now reaches U1.1 (+VOUT)
- net VDD_BUCK_5V: now also C7.1, C9.1, LDO3.2 (IN), LDO4.2 (IN), R12.1, R8.1
- net at U1.2 (TRIM): now also R1.1
- net GND: now reaches U1.3 (GND_COMMON)
- net GND: now also C1.2, C10.2, C2.2, C22.2, C3.2, C4.2, C5.2, C6.2, C7.2, C8.2, C9.2, J1.2, LDO1.3 (GND), LDO1.6 (TAB), LDO2.3 (GND), LDO2.6 (TAB), LDO3.3 (GND), LDO3.6 (TAB), LDO4.3 (GND), LDO4.6 (TAB), R1.2, R11.2, R15.2, R17.2, R2.2, R61.2, R7.2, TP13.1, TP2.1, TP4.1, TP6.1, U2.11 (EP), U2.4 (VSS), U2.6 (GND), U4.3 (GND_COMMON), U5.3 (GND_COMMON)
- net at U1.4 (+VIN): now also J1.1, U4.4 (+VIN), U5.4 (+VIN)
- new net: LDO1.5 (ADJ), R61.1, R82.2
- new net: LDO2.5 (ADJ), R5.2, R7.1
- new net: LDO3.1 (EN), R8.2
- new net: LDO3.5 (ADJ), R10.2, R11.1
- new net: R16.1, R17.1, U5.2 (TRIM)
- new net: R13.2, R14.1
- new net: R16.2, U2.2 (A)
- new net: C3.1, U2.5 (EXT_CAP)
- new net: R4.2, R5.1
- new net: LDO4.1 (EN), R12.2
- new net: LDO4.5 (ADJ), R14.2, R15.1
- new net: R60.2, R82.1
- new net: R10.1, R9.2
- new net: LDO2.1 (EN), R3.2
- new net: R2.1, U4.2 (TRIM)
- new net: LDO1.1 (EN), R59.2
- new net 1V8_ADC: C22.1, LDO1.4 (OUT), R60.1, TP14.1
- new net 1V8_Banks: C2.1, LDO2.4 (OUT), R4.1, TP1.1
- new net 2V5_IO: C8.1, LDO3.4 (OUT), R6.1, R9.1, TP3.1
- new net 3V3_IO: C10.1, C4.1, C5.1, LDO4.4 (OUT), R13.1, TP5.1, U2.1 (VDD), U2.7 (*RESET)
- new net ADDR_rheostat: U2.10 (ADDR)
- new net SCL_rheostat: U2.9 (SCL)
- new net SDA_rheostat: R6.2, U2.8 (SDA)
- new net VDD_BUCK_2V7: C1.1, C6.1, LDO1.2 (IN), LDO2.2 (IN), R3.1, R59.1, U4.1 (+VOUT)
- new net VDD_BUCK_CUSTOM: U5.1 (+VOUT)
- no-connect marks 0 -> 3
Other:
- note added: "1.8V Bank and IO Voltages (LDO)"
- note added: "1.8V to ADC"
- note added: "1.8V to Banks"
- note added: "2.5V I/O (LDO)"
- note added: "2.6897V"
- note added: "3.3V I/O (LDO)"
- note added: "Buck Voltages into LDO's"
- note added: "Cap Voltage Rating Above 7V"
- note added: "Custom Buck Voltage to DUT"
- note added: "For FIXED Voltage Operation, DNP R16 Select R17 According to the Table"
- note added: "KADC Power Rails"
- note added: "Power Plug 12V Input"
- note added: "Total 19.7k"
- note added: "Total 31.3k"
- note added: "Total 44.5k"
- note added: "Vmin = 1.735V Vtyp = 1.798V Vmax = 1.874V"
- note added: "Vmin = 2.413V Vtyp = 2.500V Vmax = 2.588V"
- note added: "Vmin = 3.19V Vtyp = 3.30V Vmax = 3.435V"
- note removed: "Power Rails to be used on the board"
- company: (none) -> The University of Chicago
- title: (none) -> KADC Power
- moved on the sheet: U1
