File: KADC_CONTROLLER/ADC.kicad_sch (KiCad schematic)
At the start: 0 parts

Commit message: Made new File for final Controller
Created a new folder "KADC_CONTROLLER_V2" which is a copy of the control board v2 schematic to increase speed. Replaced with KADC CONTROLLER components and added signals for the new pins on PSEC6
Parts:
- added C19, C20, C21, C23, C24, C25, C26, C27, C28, C29, C30, C31, C32, C33, C34, C35: 39p, symbol Device:C_Small
- added R34, R35, R36, R37, R38, R39, R40, R41, R42, R43, R44, R45, R46, R47, R48, R49: 33.2R, symbol Device:R_Small_US
- added U3, U6: AD9228ABCPZ-65, CP_48_8_ADI, symbol AD9228ABCPZ_65:AD9228ABCPZ-65
Connections:
- new net ADC_CLK1+: U3.8 (CLK+)
- new net ADC_CLK1-: U3.7 (CLK)
- new net ADC_DOUT1+: U3.20 (D_+_A)
- new net ADC_DOUT1-: U3.19 (D_-_A)
- new net ADC_DOUT2+: U3.18 (D_+_B)
- new net ADC_DOUT2-: U3.17 (D_-_B)
- new net ADC_DOUT3+: U3.16 (D_+_C)
- new net ADC_DOUT3-: U3.15 (D_-_C)
- new net ADC_DOUT4+: U3.14 (D_+_D)
- new net ADC_DOUT4-: U3.13 (D_-_D)
- new net AVDD_DUT: U3.1 (AVDD), U3.10 (AVDD), U3.2 (AVDD), U3.45 (AVDD), U3.46 (AVDD), U3.5 (AVDD), U3.6 (AVDD), U3.9 (AVDD)
- new net DCO1+: U3.24 (DCO+)
- new net DCO1-: U3.23 (DCO-)
- new net DRVDD: U3.12 (DRVDD)
- new net FCO1+: U3.22 (FCO+)
- new net FCO1-: U3.21 (FCO-)
- new net GND: C19.2, C20.2, C21.2, C23.2, C24.2, C25.2, C26.2, C27.2, C28.2, C29.2, C30.2, C31.2, C32.2, C33.2, C34.2, C35.2, U3.11 (DRGND)
- new net LPF_SIGNAL1+: C19.1, R34.2
- new net LPF_SIGNAL1-: C20.1, R35.2
- new net LPF_SIGNAL2-: C23.1, R37.2
- new net LPF_SIGNAL3+: U3.47 (VIN+C)
- new net LPF_SIGNAL3-: C25.1, R39.2, U3.48 (VIN-C)
- new net LPF_SIGNAL4+: U3.4 (VIN_+_D)
- new net LPF_SIGNAL4-: C27.1, R41.2, U3.3 (VIN__D)
- new net LPF_SIGNAL5-: C29.1, R43.2
- new net LPS_SIGNAL2+: C21.1, R36.2
- new net LPS_SIGNAL3+: C24.1, R38.2
- new net LPS_SIGNAL4+: C26.1, R40.2
- new net LPS_SIGNAL5+: C28.1, R42.2
- new net LPS_SIGNAL6+: C30.1, R44.2
- new net LPS_SIGNAL6-: C31.1, R45.2
- new net LPS_SIGNAL7+: C32.1, R46.2
- new net LPS_SIGNAL7-: C33.1, R47.2
- new net LPS_SIGNAL8+: C34.1, R48.2
- new net LPS_SIGNAL8-: C35.1, R49.2
- new net SIGNAL1+: R34.1
- new net SIGNAL1-: R35.1
- new net SIGNAL2+: R36.1
- new net SIGNAL2-: R37.1
- new net SIGNAL3+: R39.1
- new net SIGNAL3-: R38.1
- new net SIGNAL4+: R40.1
- new net SIGNAL4-: R41.1
- new net SIGNAL5+: R42.1
- new net SIGNAL5-: R43.1
- new net SIGNAL6+: R44.1
- new net SIGNAL6-: R45.1
- new net SIGNAL7+: R46.1
- new net SIGNAL7-: R47.1
- new net SIGNAL8+: R48.1
- new net SIGNAL8-: R49.1
- no-connect marks 0 -> 16
Other:
- note added: "Page Inputs"
- note added: "Page Outputs"
