File: KADC_CONTROLLER/KADC_CONTROLLER.kicad_sch (KiCad schematic)
At the start: 0 parts

Commit message: Building out New Schematic
Finished KADC Power rails, creating new Kria K26 Symbol with correct net names, SOM1 DONE. SOM2, AB DONE, CD left to do
Other:
- added sheet kria_bottom (kria_bottom.kicad_sch)
- added sheet kria_top (kria_top.kicad_sch)
- added sheet power_1 (power_1.kicad_sch)
- added sheet power_2 (power_2.kicad_sch)
- note added: "Power Rails for DUT Boards"
- note added: "Power Rails for KADC Board"
- company: (none) -> Enrico Fermi Institute - University of Chicago
- title: (none) -> Kria K26 ADC Controller (KADC)
Changed lines of the file:
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@@
 	(generator "eeschema")
 	(generator_version "9.0")
-	(paper "A4")
+	(paper "A3")
+	(title_block
+		(title "Kria K26 ADC Controller (KADC)")
+		(rev "A")
+		(company "Enrico Fermi Institute - University of Chicago")
+	)
+	(text "Power Rails for DUT Boards"
+		(exclude_from_sim no)
+		(at 75.946 15.748 0)
+		(effects
+			(font
+				(size 1.27 1.27)
+			)
+		)
+	)
+	(text "Power Rails for KADC Board"
+		(exclude_from_sim no)
+		(at 32.004 15.748 0)
+		(effects
+			(font
+				(size 1.27 1.27)
+			)
+		)
+	)
+	(sheet
+		(at 12.446 56.134)
+		(size 109.728 65.024)
+		(exclude_from_sim no)
+		(in_bom yes)
+		(on_board yes)
+		(dnp no)
+		(fields_autoplaced yes)
+		(stroke
+			(width 0.1524)
+			(type solid)
+		)
+		(fill
+			(color 0 0 0 0.0000)
+		)
+		(property "Sheetname" "kria_top"
+			(at 12.446 55.4224 0)
+			(effects
+				(font
+					(size 1.27 1.27)
+				)
+				(justify left bottom)
+			)
+		)
+		(property "Sheetfile" "kria_top.kicad_sch"
+			(at 12.446 121.7426 0)
+			(effects
+				(font
+					(size 1.27 1.27)
+				)
+				(justify left top)
+			)
+		)
+		(instances
+			(project "KADC_CONTROLLER"
+				(path "/98821545-a77c-443b-b937-4da783620b59"
+					(page "4")
+				)
+			)
+		)
+	)
+	(sheet
+		(at 12.954 20.574)
+		(size 40.894 26.416)
+		(exclude_from_sim no)
+		(in_bom yes)
+		(on_board yes)
+		(dnp no)
+		(fields_autoplaced yes)
+		(stroke
+			(width 0.1524)
+			(type solid)
+		)
+		(fill
+			(color 0 0 0 0.0000)
+		)
+		(property "Sheetname" "power_1"
+			(at 12.954 19.8624 0)
+			(effects
+				(font
+					(size 1.27 1.27)
+				)
+				(justify left bottom)
+			)
+		)
+		(property "Sheetfile" "power_1.kicad_sch"
+			(at 12.954 47.5746 0)
+			(effects
+				(font
+					(size 1.27 1.27)
+				)
+				(justify left top)
+			)
+		)
+		(instances
+			(project "KADC_CONTROLLER"
+				(path "/98821545-a77c-443b-b937-4da783620b59"
+					(page "2")
+				)
+			)
+		)
+	)
+	(sheet
+		(at 12.954 127)
+		(size 109.474 64.516)
+		(exclude_from_sim no)
+		(in_bom yes)
+		(on_board yes)
+		(dnp no)
+		(fields_autoplaced yes)
+		(stroke
+			(width 0.1524)
+			(type solid)
+		)
+		(fill
+			(color 0 0 0 0.0000)
+		)
+		(property "Sheetname" "kria_bottom"
+			(at 12.954 126.2884 0)
+			(effects
+				(font
+					(size 1.27 1.27)
+				)
+				(justify left bottom)
+			)
+		)
+		(property "Sheetfile" "kria_bottom.kicad_sch"
+			(at 12.954 192.1006 0)
+			(effects
+				(font
+					(size 1.27 1.27)
+				)
+				(justify left top)
+			)
+		)
+		(instances
+			(project "KADC_CONTROLLER"
+				(path "/98821545-a77c-443b-b937-4da783620b59"
+					(page "5")
+				)
+			)
+		)
+	)
+	(sheet
+		(at 55.88 20.32)
+		(size 41.148 26.67)
+		(exclude_from_sim no)
+		(in_bom yes)
+		(on_board yes)
+		(dnp no)
+		(fields_autoplaced yes)
+		(stroke
+			(width 0.1524)
+			(type solid)
+		)
+		(fill
+			(color 0 0 0 0.0000)
+		)
+		(property "Sheetname" "power_2"
+			(at 55.88 19.6084 0)
+			(effects
+				(font
+					(size 1.27 1.27)
+				)
+				(justify left bottom)
+			)
+		)
+		(property "Sheetfile" "power_2.kicad_sch"
+			(at 55.88 47.5746 0)
+			(effects
+				(font
+					(size 1.27 1.27)
+				)
+				(justify left top)
+			)
+		)
+		(instances
+			(project "KADC_CONTROLLER"
+				(path "/98821545-a77c-443b-b937-4da783620b59"
+					(page "3")
+				)
+			)
+		)
+	)
 	(sheet_instances
 		(path "/"
