File: KADC_CONTROLLER/kria_bottom.kicad_sch (KiCad schematic)
At the start: 0 parts

Commit message: Fixed Kria Symbol
Updated Kria symbol, fixed folders so no more problems with labeling
Parts:
- added J3: ADM6-60-01.5-L-4-2-A-TR_BOTTOM, ADM6-60-01.5-L-4-2-A-TR:SAMTEC_ADM6-60-01.5-L-4-2-A-TR, symbol AMD6_60_01_5_L_4_2_A_TR_BOTTOM:ADM6-60-01.5-L-4-2-A-TR_BOTTOM
