File: PSEC6_DUT/PSEC6_DUT_BOARD/ADC_Buffers.kicad_sch (KiCad schematic)
At the start: 0 parts

Commit message: created ADC buffer schematic
Parts:
- added C10, C12, C13, C14, C17, C19, C20, C21, C24, C26, C27, C28, C3, C31, C33, C34, C35, C38, C4, C40, C41, C42, C45, C47, C48, C49, C52, C54, C55, C56, C6, C7: 0.1u, Capacitor_SMD:C_0603_1608Metric, symbol Device:C_Small
- added C11, C16, C18, C2, C23, C25, C30, C32, C37, C39, C44, C46, C51, C53, C8, C9: 1.3p, Capacitor_SMD:C_0603_1608Metric, symbol Device:C_Small
- added C15, C22, C29, C36, C43, C5, C50, C57: 1000p, Capacitor_SMD:C_0603_1608Metric, symbol Device:C_Small
- added R10, R11, R16, R17, R22, R23, R28, R29, R34, R35, R4, R40, R41, R46, R47, R5: 2k, Resistor_SMD:R_0603_1608Metric, symbol Device:R_Small_US
- added R12, R13, R14, R15, R18, R19, R2, R20, R21, R24, R25, R26, R27, R3, R30, R31, R32, R33, R36, R37, R38, R39, R42, R43, R44, R45, R48, R49, R6, R7, R8, R9: 1000, Resistor_SMD:R_0603_1608Metric, symbol Device:R_Small_US
- added U2, U3, U4, U5, U6, U7, U8, U9: LTC6409IUDB-TRMPBF, QFN-10_UDB_LIT, symbol LTC6409IUDB:LTC6409IUDB-TRMPBF
Connections:
- new net: C53.1, R48.2, R49.2, U9.6 (-IN)
- new net: C45.1, R40.2, R41.1, U8.5 (VOCM)
- new net: C25.1, R24.2, R25.2, U5.6 (-IN)
- new net: C31.1, R28.2, R29.1, U6.5 (VOCM)
- new net: C52.1, R46.2, R47.1, U9.5 (VOCM)
- new net: C9.1, R8.2, R9.1, U3.2 (+IN)
- new net: C8.1, R6.2, R7.2, U2.6 (-IN)
- new net: C16.1, R14.2, R15.1, U4.2 (+IN)
- new net: C39.1, R36.2, R37.2, U7.6 (-IN)
- new net: C2.1, R2.1, R3.2, U2.2 (+IN)
- new net: C3.1, R4.2, R5.1, U2.5 (VOCM)
- new net: C44.1, R38.2, R39.1, U8.2 (+IN)
- new net: C46.1, R42.2, R43.2, U8.6 (-IN)
- new net: C51.1, R44.2, R45.1, U9.2 (+IN)
- new net: C32.1, R30.2, R31.2, U6.6 (-IN)
- new net: C10.1, R10.2, R11.1, U3.5 (VOCM)
- new net: C11.1, R12.2, R13.2, U3.6 (-IN)
- new net: C30.1, R26.2, R27.1, U6.2 (+IN)
- new net: C37.1, R32.2, R33.1, U7.2 (+IN)
- new net: C38.1, R34.2, R35.1, U7.5 (VOCM)
- new net: C24.1, R22.2, R23.1, U5.5 (VOCM)
- new net: C17.1, R16.2, R17.1, U4.5 (VOCM)
- new net: C18.1, R18.2, R19.2, U4.6 (-IN)
- new net: C23.1, R20.2, R21.1, U5.2 (+IN)
- new net ADC1_Out+: C8.2, R7.1, U2.7 (+OUT)
- new net ADC1_Out-: C2.2, R2.2, U2.1 (-OUT)
- new net ADC2_Out+: C11.2, R13.1, U3.7 (+OUT)
- new net ADC2_Out-: C9.2, R9.2, U3.1 (-OUT)
- new net ADC3_Out+: C18.2, R19.1, U4.7 (+OUT)
- new net ADC3_Out-: C16.2, R15.2, U4.1 (-OUT)
- new net ADC4_Out+: C25.2, R25.1, U5.7 (+OUT)
- new net ADC4_Out-: C23.2, R21.2, U5.1 (-OUT)
- new net ADC5_Out+: C32.2, R31.1, U6.7 (+OUT)
- new net ADC5_Out-: C30.2, R27.2, U6.1 (-OUT)
- new net ADC6_Out+: C39.2, R37.1, U7.7 (+OUT)
- new net ADC6_Out-: C37.2, R33.2, U7.1 (-OUT)
- new net ADC7_Out+: C46.2, R43.1, U8.7 (+OUT)
- new net ADC7_Out-: C44.2, R39.2, U8.1 (-OUT)
- new net ADC8_Out+: C53.2, R49.1, U9.7 (+OUT)
- new net ADC8_Out-: C51.2, R45.2, U9.1 (-OUT)
- new net GND: C10.2, C12.1, C13.1, C14.1, C15.1, C17.2, C19.1, C20.1, C21.1, C22.1, C24.2, C26.1, C27.1, C28.1, C29.1, C3.2, C31.2, C33.1, C34.1, C35.1, C36.1, C38.2, C4.1, C40.1, C41.1, C42.1, C43.1, C45.2, C47.1, C48.1, C49.1, C5.1, C50.1, C52.2, C54.1, C55.1, C56.1, C57.1, C6.1, C7.1, R10.1, R12.1, R16.1, R18.1, R22.1, R24.1, R28.1, R30.1, R34.1, R36.1, R4.1, R40.1, R42.1, R46.1, R48.1, R6.1, U2.10 (V-), U2.11 (V-), U2.8 (V-), U3.10 (V-), U3.11 (V-), U3.8 (V-), U4.10 (V-), U4.11 (V-), U4.8 (V-), U5.10 (V-), U5.11 (V-), U5.8 (V-), U6.10 (V-), U6.11 (V-), U6.8 (V-), U7.10 (V-), U7.11 (V-), U7.8 (V-), U8.10 (V-), U8.11 (V-), U8.8 (V-), U9.10 (V-), U9.11 (V-), U9.8 (V-)
- new net READOUT1: R3.1
- new net READOUT2: R8.1
- new net READOUT3: R14.1
- new net READOUT4: R20.1
- new net READOUT5: R26.1
- new net READOUT6: R32.1
- new net READOUT7: R38.1
- new net READOUT8: R44.1
- new net VDD18: R11.2, R17.2, R23.2, R29.2, R35.2, R41.2, R47.2, R5.2
- new net VDD33: C12.2, C13.2, C14.2, C15.2, C19.2, C20.2, C21.2, C22.2, C26.2, C27.2, C28.2, C29.2, C33.2, C34.2, C35.2, C36.2, C4.2, C40.2, C41.2, C42.2, C43.2, C47.2, C48.2, C49.2, C5.2, C50.2, C54.2, C55.2, C56.2, C57.2, C6.2, C7.2, U2.3 (*SHDN), U2.4 (V+), U2.9 (V+), U3.3 (*SHDN), U3.4 (V+), U3.9 (V+), U4.3 (*SHDN), U4.4 (V+), U4.9 (V+), U5.3 (*SHDN), U5.4 (V+), U5.9 (V+), U6.3 (*SHDN), U6.4 (V+), U6.9 (V+), U7.3 (*SHDN), U7.4 (V+), U7.9 (V+), U8.3 (*SHDN), U8.4 (V+), U8.9 (V+), U9.3 (*SHDN), U9.4 (V+), U9.9 (V+)

Commit message: DUT Board Schematic Done besides SAMTEC
The DUT Board is now done and fully documented besides the placement of the signals on the SAMTEC connector between the two boards, as the position of each connection will be determined during layout.
Connections:
- no-connect marks 0 -> 24
Other:
- note added: "From PSEC6"
- note added: "INPUTS"
- note added: "OUTPUTS"
- note added: "To Kria"
- moved on the sheet: C10, C11, C12, C13, C14, C15, C16, C17, C18, C19, C2, C20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
