File: PSEC6_DUT/PSEC6_DUT_BOARD/PSEC6_Device.kicad_sch (KiCad schematic)
At the start: 0 parts

Commit message: DUT Board Schematic Done besides SAMTEC
The DUT Board is now done and fully documented besides the placement of the signals on the SAMTEC connector between the two boards, as the position of each connection will be determined during layout.
Other:
- note added: "NOTHING TO SEE HERE"
Changed lines of the file:
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@@
 	(generator_version "10.0")
 	(paper "A4")
+	(text "NOTHING TO SEE HERE"
+		(exclude_from_sim no)
+		(at 148.336 54.356 0)
+		(effects
+			(font
+				(size 10 10)
+			)
+		)
+	)
 )
