File: KADC_CONTROLLER_V2/power.kicad_sch (KiCad schematic)
At the start: 36 parts

Commit message: many updates
Parts:
- added SW4, SW5, SW6, SW7: D6R90F2LFS, D6R90_CNK, symbol D6R90F2LFS:D6R90F2LFS
Connections:
- net GND: now also SW4.3, SW5.3, SW6.3, SW7.3; no longer C10.2, C12.2, C13.2, C8.2
- net VDD_BUCK_2V7: now also C12.2; no longer C12.1
- net VDD_BUCK_5V: now also C10.2, C8.2; no longer C10.1, C8.1
- net at LDO9.1 (EN): now also SW7.4; no longer R41.2
- net at LDO7.1 (EN): now also SW6.4; no longer R32.2
- net at LDO10.1 (EN): now also SW4.4; no longer R38.2
- net at R35.2: now also SW5.1; no longer LDO8.1 (EN)
- new net: C13.2, SW4.2
- new net: R41.2, SW7.1
- new net: C10.1, SW5.2
- new net: LDO8.1 (EN), SW5.4
- new net: C12.1, SW7.2
- new net: C8.1, SW6.2
- new net: R32.2, SW6.1
- new net: R38.2, SW4.1
Other:
- moved on the sheet: C10, C12, C13, C8, R32, R35, R38, R41

Commit message: Added footprints, updated schematic
Parts:
- SW4, SW5, SW6, SW7: footprint D6R90_CNK -> D6R90F2LFS:D6R90_CNK
Connections:
- net VDD_BUCK_5V renamed VDD_BUCK_4V
Other:
- note added: "Analog Power Rails for DUT"
Changed lines of the file:
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@@
 		)
 	)
+	(text "Analog Power Rails for DUT"
+		(exclude_from_sim no)
+		(at 97.282 20.066 0)
+		(effects
+			(font
+				(size 5 5)
+				(thickness 1)
+				(bold yes)
+				(color 0 0 0 1)
+			)
+		)
+	)
 	(text "Vmin = 1.735V\nVtyp = 1.798V\nVmax = 1.874V"
 		(exclude_from_sim no)
@@
 		)
 	)
-	(global_label "VDD_BUCK_5V"
+	(global_label "VDD_BUCK_4V"
 		(shape input)
 		(at 152.4 48.26 180)
@@
 		)
 	)
-	(global_label "VDD_BUCK_5V"
+	(global_label "VDD_BUCK_4V"
 		(shape input)
 		(at 151.13 107.95 180)
@@
 			)
 		)
-		(property "Footprint" "D6R90_CNK"
+		(property "Footprint" "D6R90F2LFS:D6R90_CNK"
 			(at 171.45 118.11 0)
 			(hide yes)
@@
 			)
 		)
-		(property "Footprint" "D6R90_CNK"
+		(property "Footprint" "D6R90F2LFS:D6R90_CNK"
 			(at 171.45 58.42 0)
 			(hide yes)
@@
 			)
 		)
-		(property "Footprint" "D6R90_CNK"
+		(property "Footprint" "D6R90F2LFS:D6R90_CNK"
 			(at 168.91 185.42 0)
 			(hide yes)
@@
 			)
 		)
-		(property "Footprint" "D6R90_CNK"
+		(property "Footprint" "D6R90F2LFS:D6R90_CNK"
 			(at 20.32 189.23 0)
 			(hide yes)
