File: KADC_CONTROLLER_V2/power2.kicad_sch (KiCad schematic)
At the start: 49 parts, among them J1 1766343, U14 OKX-T/5-D12N-C, U16 OKX-T/5-D12N-C, U17 AD5274BCPZ-100-RL7, U5 OKX-T/5-D12N-C

Commit message: many updates
Parts:
- removed C2, C3: 10u, Capacitor_SMD:C_0603_1608Metric, symbol Device:C_Small
- removed C26: 10u, symbol Device:C_Small
- removed C27: 0.1u, symbol Device:C_Small
- removed C82: 1u, symbol Device:C_Small
- removed J1: 1766343, CONN_1766343_PXC, symbol 1766343:1766343
- removed LDO2: LP38501TS-ADJ/NOPB, ul_LP38501TS-ADJ-NOPB:TS5B, symbol PSEC5_ctrlbd:LP38501TS-ADJ_NOPB
- removed R101: 10k, symbol Device:R_Small_US
- removed R11: 14.7k, Resistor_SMD:R_0603_1608Metric, symbol Device:R_Small_US
- removed R12: 4.99k, Resistor_SMD:R_0603_1608Metric, symbol Device:R_Small_US
- removed R13, R8: 10k, Resistor_SMD:R_0603_1608Metric, symbol Device:R_Small_US
- removed R29: FIXED, symbol Device:R_Small_US
- removed R44: 0R, symbol Device:R_Small_US
- removed TP10: GND, TestPoint:TestPoint_THTPad_1.5x1.5mm_Drill0.7mm, symbol Connector:TestPoint
- removed TP9: 1V8_Bank, TestPoint:TestPoint_THTPad_1.5x1.5mm_Drill0.7mm, symbol Connector:TestPoint
- removed U16: OKX-T/5-D12N-C, OKX-T/5-D12N-C_MUR, symbol OKX_T_5_D12N_C:OKX-T_5-D12N-C
- removed U17: AD5274BCPZ-100-RL7, CP_10_9_ADI, symbol AD5274BCPZ_100_RL7:AD5274BCPZ-100-RL7
Connections:
- net 1V8_ADC: no longer C22.1, LDO1.4 (OUT), R60.1, TP14.1
- net 2V5_IO: no longer C23.1, LDO3.4 (OUT), R45.1, TP16.1
- net 3V3_IO: no longer C95.1, LDO4.4 (OUT), R102.1, TP21.1
- net 12V_IN: now reaches U14.4 (+VIN), U5.4 (+VIN)
- new net 1V8_PERI: C22.1, LDO1.4 (OUT), R60.1, TP14.1
- new net 2V5_PERI: C23.1, LDO3.4 (OUT), R45.1, TP16.1
- new net 3V3_PERI: C95.1, LDO4.4 (OUT), R102.1, TP21.1
- no-connect marks 13 -> 12
Other:
- note added: "1.8V to Peripheral Devices"
- note added: "2.5V Peripheral Devices"
- note added: "3.3V Peripheral Devices"
- note added: "Analog Power Rails for Peripherals and DUT"
- note removed: "1.8V Bank and IO Voltages (LDO)"
- note removed: "1.8V to ADC"
- note removed: "1.8V to Banks"
- note removed: "2.5V I/O (LDO)"
- note removed: "3.3V I/O (LDO)"
- note removed: "Cap Voltage Rating Above 7V"
- note removed: "Custom Buck Voltage to DUT"
- note removed: "For FIXED Voltage Operation, DNP R16 Select R17 According to the Table"
- note removed: "KADC Power Rails"
- note removed: "Power Plug 12V Input"
- moved on the sheet: C14, C22, LDO1, R10, R2, R59, R60, R61, R82, TP13, TP14, U14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

Commit message: Added footprints, updated schematic
Parts:
- added SW10, SW8, SW9: D6R90F2LFS, D6R90F2LFS:D6R90_CNK, symbol D6R90F2LFS:D6R90F2LFS
- R10: value 1.47k -> 2.21k
- U14, U5: footprint OKX-T/5-D12N-C_MUR -> OKX_T_5_D12N_C:OKX-T&slash_5-D12N-C_MUR
Connections:
- net GND: now also SW10.3, SW8.3, SW9.3; no longer C14.2, C15.2, C94.2
- net VDD_BUCK_2V7: now also C14.2; no longer C14.1
- net at R14.2: now also SW9.1; no longer LDO3.1 (EN)
- net at R85.2: now also SW10.1; no longer LDO4.1 (EN)
- net at R59.2: now also SW8.1; no longer LDO1.1 (EN)
- net VDD_BUCK_5V renamed VDD_BUCK_4V
- net VDD_BUCK_4V: now also C15.2, C94.2; no longer C15.1, C94.1
- new net: C14.1, SW8.2
- new net: C94.1, SW10.2
- new net: LDO1.1 (EN), SW8.4
- new net: LDO4.1 (EN), SW10.4
- new net: LDO3.1 (EN), SW9.4
- new net: C15.1, SW9.2
- no-connect marks 12 -> 2
Other:
- note added: "Analog Power Rails for Peripherals"
- note added: "At 2.21k VOUT = 4.023V"
- note removed: "12V Plug"
- note removed: "Analog Power Rails for Peripherals and DUT"
- note removed: "Page Inputs"
- note removed: "Page Outputs"
- moved on the sheet: C14, C15, C94, R14, R59, R85
