File: KADC_CONTROLLER_V2/DisplayPort.kicad_sch (KiCad schematic)
At the start: 32 parts, among them J11 472720001, U1 SN74AVC2T245RSWR, U54 SN74AVC2T245RSWR, U55 FIN1019MTCX, U56 STMPS2151STR, U57 TPD8S009DSMR

Commit message: More Things
Parts:
- added R206, R207: 1M, Resistor_SMD:R_0603_1608Metric, symbol Device:R_Small_US
Connections:
- net GND: now also R206.2, R207.2
- net at J11.13: now also R206.1
- net at J11.14: now also R207.1

Commit message: Quick Updates, Power verification finalized
Parts:
- J11: footprint CONN_47272-0001_MOL -> 47270001:CONN_47272-0001_MOL
- U1, U54: footprint RSW0010A -> SN74AVC2T245RSWR:RSW0010A
- U55: footprint TSSOP14_4P4X5_ONS -> FIN1019MTCX:TSSOP14_4P4X5_ONS
- U56: footprint SOT23-5L_STM -> STMPS215STR:SOT23-5L_STM
- U57: footprint DSM15_X -> TPD8S009DSMR:DSM15_X
Changed lines of the file:
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@@
 			)
 		)
-		(property "Footprint" "SOT23-5L_STM"
+		(property "Footprint" "STMPS215STR:SOT23-5L_STM"
 			(at 478.028 93.218 0)
 			(hide yes)
@@
 			)
 		)
-		(property "Footprint" "CONN_47272-0001_MOL"
+		(property "Footprint" "47270001:CONN_47272-0001_MOL"
 			(at 258.572 239.522 0)
 			(hide yes)
@@
 			)
 		)
-		(property "Footprint" "TSSOP14_4P4X5_ONS"
+		(property "Footprint" "FIN1019MTCX:TSSOP14_4P4X5_ONS"
 			(at 241.046 101.346 0)
 			(hide yes)
@@
 			)
 		)
-		(property "Footprint" "DSM15_X"
+		(property "Footprint" "TPD8S009DSMR:DSM15_X"
 			(at 472.186 181.864 0)
 			(hide yes)
@@
 			)
 		)
-		(property "Footprint" "RSW0010A"
+		(property "Footprint" "SN74AVC2T245RSWR:RSW0010A"
 			(at 149.86 179.07 0)
 			(hide yes)
@@
 			)
 		)
-		(property "Footprint" "RSW0010A"
+		(property "Footprint" "SN74AVC2T245RSWR:RSW0010A"
 			(at 149.86 104.14 0)
 			(hide yes)
