File: KADC_CONTROLLER_V2/ethernet.kicad_sch (KiCad schematic)
At the start: 46 parts, among them Q6 2N7002BK,215, Q8 2N7002BK,215, T1 7499111446, U1 88E1512-A0-NNP2C000, Y1 ECS-3225MV-250-BN-TR3

Commit message: many updates
Parts:
- removed C106, C118, C17, C21, C46, C48, C49, C50, C51, C58, C61, C63: 470n, Capacitor_SMD:C_0603_1608Metric, symbol Device:C
- removed C119, C52: 4.7u, Capacitor_SMD:C_0603_1608Metric, symbol Device:C
- removed C155: 470n, Capacitor_SMD:C_0603_1608Metric, symbol Device:C_Small
- removed C5: 10n, Capacitor_SMD:C_0603_1608Metric, symbol Device:C
- removed C53, C54, C55, C56, C62, C64: 100n, Capacitor_SMD:C_0603_1608Metric, symbol Device:C
- removed C57: 47p, Capacitor_SMD:C_0603_1608Metric, symbol Device:C
- removed C59: 100u, Capacitor_SMD:C_0805_2012Metric, symbol Device:C
- removed L3: 220R @ 100mHz, Resistor_SMD:R_0402_1005Metric, symbol Device:L
- removed L5: 220R@100MHz, Resistor_SMD:R_0603_1608Metric, symbol Device:L
- removed Q6, Q8: 2N7002BK,215, SI2342DS_T1_GE3:SOT-23_TO-236_VIS, symbol Simulation_SPICE:NMOS
- removed R100: 1M2, Resistor_SMD:R_0603_1608Metric, symbol Device:R_US
- removed R112, R113: 10k, Resistor_SMD:R_0603_1608Metric, symbol Device:R_Small_US
- removed R114, R115: 0R, Resistor_SMD:R_0603_1608Metric, symbol Device:R_Small_US
- removed R22: 4k99, Resistor_SMD:R_0603_1608Metric, symbol Device:R_US
- removed R23, R24, R26, R27, R28, R78: 22, Resistor_SMD:R_0603_1608Metric, symbol Device:R_US
- removed R74, R76: 240R, Resistor_SMD:R_0603_1608Metric, symbol Device:R_Small_US
- removed R84: 10k, Resistor_SMD:R_0603_1608Metric, symbol Device:R_US
- removed T1: 7499111446, Connector_RJ:RJ45_Wuerth_7499111446_Horizontal, symbol PSEC5_ctrlbd:WE-RJ45_7499111446
- removed U1: 88E1512-A0-NNP2C000, QFN_56P_MTG, symbol PSEC5_ctrlbd:88E1512-A0-NNP2C000
- removed Y1: ECS-3225MV-250-BN-TR3, ECS-3225MV-250-BN-TR3:OSC_ECS-2333-160-BN-TR, symbol Oscillator:ECS-3225MV-250-BN-TR3
- added C199, C200, C201, C207, C208, C213, C214, C215, C216, C225, C226, C227, C228: 0.1u, Capacitor_SMD:C_0603_1608Metric, symbol Device:C_Small
- added C202, C212, C221: 0.01u, Capacitor_SMD:C_0603_1608Metric, symbol Device:C_Small
- added C203, C204, C205, C209, C210, C217, C218, C219, C220: 1u, Capacitor_SMD:C_0603_1608Metric, symbol Device:C_Small
- added C206, C211, C222: 10u, Capacitor_SMD:C_0603_1608Metric, symbol Device:C_Small
- added C223, C224: 27p, Capacitor_SMD:C_0603_1608Metric, symbol Device:C_Small
- added Q5, Q7, Q9: DMN2310U-7, Package_TO_SOT_SMD:TSOT-23, symbol Simulation_SPICE:NMOS
- added R180, R192: 10k, Resistor_SMD:R_0603_1608Metric, symbol Device:R_Small_US
- added R181, R182, R183: 4.7k, Resistor_SMD:R_0603_1608Metric, symbol Device:R_Small_US
- added R184: 11k, Resistor_SMD:R_0603_1608Metric, symbol Device:R_Small_US
- added R185, R186, R187, R188, R189, R191, R193, R194, R195, R196, R197, R199: DNP, Resistor_SMD:R_0603_1608Metric, symbol Device:R_Small_US
- added R190: 5.76k, Resistor_SMD:R_0603_1608Metric, symbol Device:R_Small_US
- added R198, R200: 2.49k, Resistor_SMD:R_0603_1608Metric, symbol Device:R_Small_US
- added R201, R202: 2.21k, Resistor_SMD:R_0603_1608Metric, symbol Device:R_Small_US
- added U52: L829-1J1T-43, L829-1J1T-43_BEL, symbol L829_1J1T_43:L829-1J1T-43
- added U53: DP83867CRRGZR, RGZ0048B, symbol DP83867CRRGZR:DP83867CRRGZR
Connections:
- net GND: now also C199.2, C200.2, C201.2, C202.2, C203.2, C204.2, C205.2, C206.2, C207.2, C208.2, C209.2, C210.2, C211.2, C212.2, C213.2, C214.2, C215.2, C216.2, C217.2, C218.2, C219.2, C220.2, C221.2, C222.2, C224.1, C225.1, C226.1, C227.1, C228.1, Q5.3 (S), Q7.3 (S), Q9.3 (S), R184.2, R193.2, R194.2, R195.2, R196.2, R197.2, R198.2, R199.2, R200.2, U53.49 (PAD)
- new net: R180.2, U53.43 (RESET_N)
- new net: R183.2, U53.22 (JTAG_TMS)
- new net: C225.2, U52.12 (TRCT0)
- new net: R185.1, R186.1, R187.1, R188.1, R189.1, R190.1, R191.1, R192.1
- new net: R182.2, U53.20 (JTAG_CLK)
- new net: C223.1, C224.2, U53.15 (X_I)
- new net: R181.2, U53.23 (JTAG_TDI)
- new net: C227.2, U52.1 (TRCT2)
- new net: C226.2, U52.6 (TRCT1)
- new net: C228.2, U52.7 (TRCT3)
- new net: R184.1, U53.12 (RBIAS)
- new net: R201.2, U53.44 (INT_PWDN)
- new net ETH_1V0: C213.1, C214.1, C215.1, C216.1, C217.1, C218.1, C219.1, C220.1, C221.1, C222.1, U53.24 (VDD1P0), U53.31 (VDD1P0), U53.42 (VDD1P0), U53.6 (VDD1P0)
- new net ETH_2V5: C207.1, C208.1, C209.1, C210.1, C211.1, C212.1, U53.3 (VDDA2P5), U53.9 (VDDA2P5)
- new net GEM3_MDC: U53.16 (MDC)
- new net GEM3_MDIO: R202.2, U53.17 (MDIO)
- new net GEM_GPIO0: R186.2, R194.1, U53.39 (GPIO_0)
- new net GEM_GPIO1: R185.2, R193.1, U53.40 (GPIO_1)
- new net GEM_LED0: Q9.2 (G), R189.2, R197.1, U53.47 (LED_0)
- new net GEM_LED0_CA: Q9.1 (D), U52.15 (LEFT_ORG_CA)
- new net GEM_LED1: Q7.2 (G), R188.2, R196.1, U53.46 (LED_1)
- new net GEM_LED1_CA: Q7.1 (D), U52.17 (LEFT_GRN_CA)
- new net GEM_LED2: Q5.2 (G), R187.2, R195.1, U53.45 (LED_2)
- new net GEM_LED2_CA: Q5.1 (D), U52.13 (RIGHT_YLW_CA)
- new net GEM_TD_A_N: U52.10 (TD0_N), U53.2 (TD_M_A)
- new net GEM_TD_A_P: U52.11 (TD0_P), U53.1 (TD_P_A)
- new net GEM_TD_B_N: U52.5 (TD1_N), U53.5 (TD_M_B)
- new net GEM_TD_B_P: U52.4 (TD1_P), U53.4 (TD_P_B)
- new net GEM_TD_C_N: U52.2 (TD2_N), U53.8 (TD_M_C)
- new net GEM_TD_C_P: U52.3 (TD2_P), U53.7 (TD_P_C)
- new net GEM_TD_D_N: U52.9 (TD3_N), U53.11 (TD_M_D)
- new net GEM_TD_D_P: U52.8 (TD3_P), U53.10 (TD_P_D)
- new net PS_1V8: C199.1, C200.1, C201.1, C202.1, C203.1, C204.1, C205.1, C206.1, R180.1, R181.1, R182.1, R183.1, R201.1, R202.1, U53.19 (VDDIO), U53.30 (VDDIO), U53.41 (VDDIO)
- new net PS_3V3: U52.14 (RIGHT_YLW_AN), U52.16 (LEFT_GRNORG_AN)
- new net RGMII_RX_CLK: U53.32 (RX_CLK)
- new net RGMII_RX_CTL: R190.2, R198.1, U53.38 (RX_DV_RX_CTRL)
- new net RGMII_RX_D0: R192.2, R200.1, U53.33 (RX_D0)
- new net RGMII_RX_D1: U53.34 (RX_D1)
- new net RGMII_RX_D2: R191.2, R199.1, U53.35 (RX_D2)
- new net RGMII_RX_D3: U53.36 (RX_D3)
- new net RGMII_TX_CLK: U53.29 (GTX_CLK)
- new net RGMII_TX_CTL: U53.37 (TX_EN_TX_CTRL)
- new net RGMII_TX_D0: U53.28 (TX_D0)
- new net RGMII_TX_D1: U53.27 (TX_D1)
- new net RGMII_TX_D2: U53.26 (TX_D2)
- new net RGMII_TX_D3: U53.25 (TX_D3)
- no-connect marks 10 -> 5
Other:
- note added: "50VDC"
- note added: "ADDR = 0x01"
- note added: "MIO 64"
- note added: "MIO 65"
- note added: "MIO 66"
- note added: "MIO 67"
- note added: "MIO 68"
- note added: "MIO 69"
- note added: "MIO 70"
- note added: "MIO 71"
- note added: "MIO 72"
- note added: "MIO 73"
- note added: "MIO 74"
- note added: "MIO 75"
- note added: "MIO 76"
- note added: "MIO 77"
- note added: "MIO GEM3"
- note removed: "742863122"

Commit message: More Things
Connections:
- net PS_POR: now reaches R180.2, U53.43 (RESET_N)
- net ETH_REF_CLK: now reaches C223.2
Changed lines of the file:
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@@
+		)
+	)
+	(global_label "ETH_REF_CLK"
+		(shape input)
+		(at 396.24 283.21 0)
+		(fields_autoplaced yes)
+		(effects
+			(font
+				(size 1.27 1.27)
+			)
+			(justify left)
+		)
+		(property "Intersheetrefs" "${INTERSHEET_REFS}"
+			(at 411.6832 283.21 0)
+			(hide yes)
+			(show_name no)
+			(do_not_autoplace no)
+			(effects
+				(font
+					(size 1.27 1.27)
+				)
+				(justify left)
+			)
 		)
 	)
@@
 			)
 		)
+	)
+	(global_label "PS_POR"
+		(shape input)
+		(at 194.31 303.53 180)
+		(fields_autoplaced yes)
+		(effects
+			(font
+				(size 1.27 1.27)
+			)
+			(justify right)
+		)
+		(property "Intersheetrefs" "${INTERSHEET_REFS}"
+			(at 184.0072 303.53 0)
+			(hide yes)
+			(show_name no)
+			(do_not_autoplace no)
+			(effects
+				(font
+					(size 1.27 1.27)
+				)
+				(justify right)
+			)
+		)

Commit message: Added footprints, updated schematic
Connections:
- net PS_1V8: now also R185.1, R186.1, R187.1, R188.1, R189.1, R190.1, R191.1, R192.1
Changed lines of the file:
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@@
-	(wire
-		(pts
-			(xy 69.85 212.09) (xy 69.85 220.98)
-		)
-		(stroke
-			(width 0)
-			(type default)
-		)
-	)
 	(wire
 		(pts
@@
 		)
 		(stroke
+			(width 0)
+			(type default)
+		)
+	)
+	(wire
+		(pts
+			(xy 69.85 210.82) (xy 69.85 220.98)
+		)
+		(stroke

Commit message: Quick Updates, Power verification finalized
Parts:
- removed Q5, Q7, Q9: DMN2310U-7, Package_TO_SOT_SMD:TSOT-23, symbol Simulation_SPICE:NMOS
- added Q16, Q17, Q18: BSS806NEH6327XTSA1, Package_TO_SOT_SMD:SOT-23-3, symbol Transistor_FET:Q_NMOS_GSD
- U52: footprint L829-1J1T-43_BEL -> L829_1J1T_43:L829-1J1T-43_BEL
- U53: footprint RGZ0048B -> DP83867CRRGZR:RGZ0048B
Connections:
- net GEM_LED0: now also Q18.1 (G)
- net GEM_LED0_CA: now also Q18.3 (D)
- net GEM_LED1: now also Q17.1 (G)
- net GEM_LED1_CA: now also Q17.3 (D)
- net GEM_LED2: now also Q16.1 (G)
- net GEM_LED2_CA: now also Q16.3 (D)
- net GND: now also Q16.2 (S), Q17.2 (S), Q18.2 (S)
