File: KADC_CONTROLLER_V2/untitled.SOM240_1(1.5).kicad_sch (KiCad schematic)
At the start: 24 parts, among them J10 ADM6-60-01.5-L-4-2-A-TR, J7 1766453, SW2 SW_MEC_5G

Commit message: many updates
Parts:
- removed C70, C71: 100n, Capacitor_SMD:C_0603_1608Metric, symbol Device:C_Small
- removed J7: 1766453, 1766453:CONN_1766453, symbol PSEC5_ctrlbd:1766453
Connections:
- net UART_CTS: no longer J10.C30 (MIO29)
- net UART_RTS: no longer J10.C31 (MIO30)
- net VCCOEN_PS_M2C: now reaches J10.A19 (VCCOEN_PS_M2C)
- net VCCOEN_PL_M2C: now reaches J10.A20 (VCCOEN_PL_M2C)
- net USB0_DATA5: now reaches J10.A38 (MIO61)
- net USB0_DATA6: now reaches J10.A39 (MIO62)
- net USB0_DATA7: now reaches J10.A40 (MIO63)
- net GTR_DP1_M2C_P: now reaches J10.A47 (GTR_DP1_M2C_P)
- net GTR_DP1_M2C_N: now reaches J10.A48 (GTR_DP1_M2C_N)
- net USB0_STP: now reaches J10.B40 (MIO58)
- net USB0_DATA3: now reaches J10.B41 (MIO59)
- net USB0_DATA4: now reaches J10.B42 (MIO60)
- net GTR_DP2_C2M_P: now reaches J10.B53 (GTR_DP2_C2M_P)
- net GTR_DP2_C2M_N: now reaches J10.B54 (GTR_DP2_C2M_N)
- net USB0_NXT: now reaches J10.C38 (MIO55)
- net USB0_DATA0: now reaches J10.C39 (MIO56)
- net USB0_DATA1: now reaches J10.C40 (MIO57)
- net MIO27: now reaches J10.D29 (MIO27)
- net MIO28: now reaches J10.D30 (MIO28)
- net USB0_CLK: now reaches J10.D36 (MIO52)
- net USB0_DIR: now reaches J10.D37 (MIO53)
- net USB0_DATA2: now reaches J10.D38 (MIO54)
- net GTR_DP2_M2C_P: now reaches J10.D57 (GTR_DP2_M2C_P)
- net GTR_DP2_M2C_N: now reaches J10.D58 (GTR_DP2_M2C_N)
- net 1V8_Banks renamed PL_1V8
- net 2V5_IO renamed PL_2V5
- net VDD_BUCK_5V renamed 5V0_IN
- new net MIO29: J10.C30 (MIO29)
- new net MIO30: J10.C31 (MIO30)
- no-connect marks 60 -> 38
Other:
- added sheet DisplayPort (DisplayPort.kicad_sch)
- added sheet i2c (i2c.kicad_sch)
- sheet USB-UART1 ports: added USB0_CLK, USB0_DATA0, USB0_DATA1, USB0_DATA2, USB0_DATA3, USB0_DATA4, USB0_DATA5, USB0_DATA6, USB0_DATA7, USB0_DIR, USB0_NXT, USB0_STP; removed none
- note removed: "Vertical 2 pin Connector for Kria Fan"

Commit message: More Things
Connections:
- net GTR_REFCLK1_C2M_P: now reaches J10.B49 (GTR_REFCLK1_C2M_P)
- net GTR_REFCLK1_C2M_N: now reaches J10.B50 (GTR_REFCLK1_C2M_N)
- net GTR_REFCLK0_C2M_P: now reaches J10.C47 (GTR_REFCLK0_C2M_P)
- net GTR_REFCLK0_C2M_N: now reaches J10.C48 (GTR_REFCLK0_C2M_N)
- net GTR_REFCLK2_C2M_P: now reaches J10.D53 (GTR_REFCLK2_C2M_P)
- net GTR_REFCLK2_C2M_N: now reaches J10.D54 (GTR_REFCLK2_C2M_N)
- no-connect marks 38 -> 32
Changed lines of the file:
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@@
 	)
 	(no_connect
-		(at 121.92 146.05)
-	)
-	(no_connect
-		(at 214.63 142.24)
-	)
-	(no_connect
 		(at 121.92 72.39)
 	)
 	(no_connect
-		(at 121.92 143.51)
-	)
-	(no_connect
 		(at 121.92 100.33)
 	)
@@
 	)
 	(no_connect
-		(at 251.46 157.48)
-	)
-	(no_connect
 		(at 121.92 105.41)
 	)
@@
 	)
 	(no_connect
-		(at 251.46 154.94)
-	)
-	(no_connect
 		(at 121.92 90.17)
 	)
@@
 	)
 	(no_connect
-		(at 214.63 139.7)
-	)
-	(no_connect
 		(at 80.01 161.29)
 	)
@@
 	(wire
 		(pts
+			(xy 200.66 142.24) (xy 214.63 142.24)
+		)
+		(stroke
+			(width 0)
+			(type default)
+		)
+	)
+	(wire
+		(pts
+			(xy 121.92 146.05) (xy 130.81 146.05)
+		)
+		(stroke
+			(width 0)
+			(type default)
+		)
+	)
+	(wire
+		(pts
 			(xy 76.2 146.05) (xy 80.01 146.05)
 		)
@@
 	(wire
 		(pts
+			(xy 251.46 154.94) (xy 265.43 154.94)
+		)
+		(stroke
+			(width 0)
+			(type default)
+		)
+	)
+	(wire
+		(pts
 			(xy 121.92 21.59) (xy 144.78 21.59)
 		)
@@
 	(wire
 		(pts
+			(xy 121.92 143.51) (xy 130.81 143.51)
+		)
+		(stroke
+			(width 0)
+			(type default)
+		)
+	)
+	(wire
+		(pts
 			(xy 191.77 27.94) (xy 214.63 27.94)
 		)
@@
 	(wire
 		(pts
+			(xy 251.46 157.48) (xy 265.43 157.48)
+		)
+		(stroke
+			(width 0)
+			(type default)
+		)
+	)
+	(wire
+		(pts
 			(xy 76.2 135.89) (xy 76.2 143.51)
 		)
@@
 	(wire
 		(pts
+			(xy 200.66 139.7) (xy 214.63 139.7)
+		)
+		(stroke
+			(width 0)
+			(type default)
+		)
+	)
+	(wire
+		(pts
 			(xy 255.27 43.18) (xy 255.27 50.8)
 		)
@@
 		)
 	)
+	(global_label "GTR_REFCLK1_C2M_P"
+		(shape input)
+		(at 130.81 143.51 0)
+		(fields_autoplaced yes)
+		(effects
+			(font
+				(size 1.27 1.27)
+			)
+			(justify left)
+		)
+		(property "Intersheetrefs" "${INTERSHEET_REFS}"
+			(at 153.6917 143.51 0)
+			(hide yes)
+			(show_name no)
+			(do_not_autoplace no)
+			(effects
+				(font
+					(size 1.27 1.27)
+				)
+				(justify left)
+			)
+		)
+	)
 	(global_label "GTR_DP2_C2M_P"
 		(shape output)
@@
 		)
 	)
+	(global_label "GTR_REFCLK1_C2M_N"
+		(shape input)
+		(at 130.81 146.05 0)
+		(fields_autoplaced yes)
+		(effects
+			(font
+				(size 1.27 1.27)
+			)
+			(justify left)
+		)
+		(property "Intersheetrefs" "${INTERSHEET_REFS}"
+			(at 153.7522 146.05 0)
+			(hide yes)
+			(show_name no)
+			(do_not_autoplace no)
+			(effects
+				(font
+					(size 1.27 1.27)
+				)
+				(justify left)
+			)
+		)
+	)
 	(global_label "SPIclk"
 		(shape input)
@@
 		)
 	)
+	(global_label "GTR_REFCLK0_C2M_N"
+		(shape input)
+		(at 200.66 142.24 180)
+		(fields_autoplaced yes)
+		(effects
+			(font
+				(size 1.27 1.27)
+			)
+			(justify right)
+		)
+		(property "Intersheetrefs" "${INTERSHEET_REFS}"
+			(at 177.7178 142.24 0)
+			(hide yes)
+			(show_name no)
+			(do_not_autoplace no)
+			(effects
+				(font
+					(size 1.27 1.27)
+				)
+				(justify right)
+			)
+		)
+	)
+	(global_label "GTR_REFCLK0_C2M_P"
+		(shape input)
+		(at 200.66 139.7 180)
+		(fields_autoplaced yes)
+		(effects
+			(font
+				(size 1.27 1.27)
+			)
+			(justify right)
+		)
+		(property "Intersheetrefs" "${INTERSHEET_REFS}"
+			(at 177.7783 139.7 0)
+			(hide yes)
+			(show_name no)
+			(do_not_autoplace no)
+			(effects
+				(font
+					(size 1.27 1.27)
+				)
+				(justify right)
+			)
+		)
+	)
+	(global_label "GTR_REFCLK2_C2M_N"
+		(shape input)
+		(at 265.43 157.48 0)
+		(fields_autoplaced yes)
+		(effects
+			(font
+				(size 1.27 1.27)
+			)
+			(justify left)
+		)
+		(property "Intersheetrefs" "${INTERSHEET_REFS}"
+			(at 288.3722 157.48 0)
+			(hide yes)
+			(show_name no)
+			(do_not_autoplace no)
+			(effects
+				(font
+					(size 1.27 1.27)
+				)
+				(justify left)
+			)
+		)
+	)
 	(global_label "5V0_IN"
 		(shape input)
@@
 			)
 		)
+	)
+	(global_label "GTR_REFCLK2_C2M_P"
+		(shape input)
+		(at 265.43 154.94 0)
+		(fields_autoplaced yes)
+		(effects
+			(font
+				(size 1.27 1.27)
+			)
+			(justify left)
+		)
+		(property "Intersheetrefs" "${INTERSHEET_REFS}"
+			(at 288.3117 154.94 0)
+			(hide yes)
+			(show_name no)
+			(do_not_autoplace no)
+			(effects
+				(font
+					(size 1.27 1.27)
+				)
+				(justify left)
+			)
+		)

Commit message: quick changes
Connections:
- net I2C_SCK: now reaches J10.C26 (MIO24_I2C_SCK)
- net I2C_SDA: now reaches J10.C27 (MIO25_I2C_SDA)
- net ETH_MDC renamed GEM3_MDC
- net ETH_MDIO renamed GEM3_MDIO
- net ETH_RXD0 renamed RGMII_RX_D0
- net ETH_RXD1 renamed RGMII_RX_D1
- net ETH_RXD2 renamed RGMII_RX_D2
- net ETH_RXD3 renamed RGMII_RX_D3
- net ETH_RX_CLK renamed RGMII_RX_CLK
- net ETH_RX_CTRL renamed RGMII_RX_CTL
- net ETH_TXD0 renamed RGMII_TX_D0
- net ETH_TXD1 renamed RGMII_TX_D1
- net ETH_TXD2 renamed RGMII_TX_D2
- net ETH_TXD3 renamed RGMII_TX_D3
- net ETH_TX_CLK renamed RGMII_TX_CLK
- net ETH_TX_CTRL renamed RGMII_TX_CTL
- no-connect marks 32 -> 30
Other:
- sheet ethernet1 ports: added GEM3_MDC, GEM3_MDIO, RGMII_RX_CLK, RGMII_RX_CTL, RGMII_RX_D0, RGMII_RX_D1, RGMII_RX_D2, RGMII_RX_D3, RGMII_TX_CLK, RGMII_TX_CTL, RGMII_TX_D0, RGMII_TX_D1, RGMII_TX_D2, RGMII_TX_D3; removed ETH_MDC, ETH_MDIO, ETH_RXD0, ETH_RXD1, ETH_RXD2, ETH_RXD3, ETH_RX_CLK, ETH_RX_CTRL, ETH_TXD0, ETH_TXD1, ETH_TXD2, ETH_TXD3, ETH_TX_CLK, ETH_TX_CTRL

Commit message: Added footprints, updated schematic
Parts:
- removed R1, R3, R4, R5, R6, R7: 22R 1%, Resistor_SMD:R_0603_1608Metric, symbol Device:R_US
- removed R70, R71, R73, R75: DNP, Resistor_SMD:R_0603_1608Metric, symbol Device:R_Small_US
- added S1: DS01C-254-S-04BE, DS01C-254-S-04BE:SW_DS01C-254-S-04BE, symbol DS01C-254-S-04BE:DS01C-254-S-04BE
Connections:
- net GND: now also S1.1B, S1.2B, S1.3B, S1.4B
- net MODE0: now also S1.1A
- net MODE1: now also S1.2A
- net MODE2: now also S1.3A
- net MODE3: now also S1.4A
- net RGMII_TX_CLK: now also J10.D40 (MIO64)
- net RGMII_TX_CTL: now also J10.C44 (MIO69)
- net RGMII_TX_D0: now also J10.D41 (MIO65)
- net RGMII_TX_D1: now also J10.D42 (MIO66)
- net RGMII_TX_D2: now also J10.C42 (MIO67)
- net RGMII_TX_D3: now also J10.C43 (MIO68)
- net PWROFF_C2M_B: now reaches J10.B26 (PWROFF_C2M_L), TP30.1
Other:
- moved on the sheet: TP12, TP29, TP30

Commit message: Added SOM dedicated power rail
Connections:
- net 5V0_IN renamed 5V0_SOM
Changed lines of the file:
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@@
+		)
+	)
+	(global_label "5V0_SOM"
+		(shape input)
+		(at 142.24 171.45 0)
+		(fields_autoplaced yes)
+		(effects
+			(font
+				(size 1.27 1.27)
+			)
+			(justify left)
+		)
+		(property "Intersheetrefs" "${INTERSHEET_REFS}"
+			(at 153.6918 171.45 0)
+			(hide yes)
+			(show_name no)
+			(do_not_autoplace no)
+			(effects
+				(font
+					(size 1.27 1.27)
+				)
+				(justify left)
+			)
 		)
 	)
@@
 		)
 	)
-	(global_label "5V0_IN"
+	(global_label "PS_SRST"
+		(shape input)
+		(at 193.04 60.96 180)
+		(fields_autoplaced yes)
+		(effects
+			(font
+				(size 1.27 1.27)
+			)
+			(justify right)
+		)
+		(property "Intersheetrefs" "${INTERSHEET_REFS}"
+			(at 181.9511 60.96 0)
+			(hide yes)
+			(show_name no)
+			(do_not_autoplace no)
+			(effects
+				(font
+					(size 1.27 1.27)
+				)
+				(justify right)
+			)
+		)
+	)
+	(global_label "5V0_SOM"
+		(shape input)
+		(at 265.43 172.72 0)
+		(fields_autoplaced yes)
+		(effects
+			(font
+				(size 1.27 1.27)
+			)
+			(justify left)
+		)
+		(property "Intersheetrefs" "${INTERSHEET_REFS}"
+			(at 276.8818 172.72 0)
+			(hide yes)
+			(show_name no)
+			(do_not_autoplace no)
+			(effects
+				(font
+					(size 1.27 1.27)
+				)
+				(justify left)
+			)
+		)
+	)
+	(global_label "GTR_REFCLK0_C2M_N"
+		(shape input)
+		(at 200.66 142.24 180)
+		(fields_autoplaced yes)
+		(effects
+			(font
+				(size 1.27 1.27)
+			)
+			(justify right)
+		)
+		(property "Intersheetrefs" "${INTERSHEET_REFS}"
+			(at 177.7178 142.24 0)
+			(hide yes)
+			(show_name no)
+			(do_not_autoplace no)
+			(effects
+				(font
+					(size 1.27 1.27)
+				)
+				(justify right)
+			)
+		)
+	)
+	(global_label "GTR_REFCLK0_C2M_P"
+		(shape input)
+		(at 200.66 139.7 180)
+		(fields_autoplaced yes)
+		(effects
+			(font
+				(size 1.27 1.27)
+			)
+			(justify right)
+		)
+		(property "Intersheetrefs" "${INTERSHEET_REFS}"
+			(at 177.7783 139.7 0)
+			(hide yes)
+			(show_name no)
+			(do_not_autoplace no)
+			(effects
+				(font
+					(size 1.27 1.27)
+				)
+				(justify right)
+			)
+		)
+	)
+	(global_label "5V0_SOM"
 		(shape input)
 		(at 200.66 171.45 180)
@@
 		)
 		(property "Intersheetrefs" "${INTERSHEET_REFS}"
-			(at 191.2643 171.45 0)
-			(hide yes)
-			(show_name no)
-			(do_not_autoplace no)
-			(effects
-				(font
-					(size 1.27 1.27)
-				)
-				(justify right)
-			)
-		)
-	)
-	(global_label "5V0_IN"
-		(shape input)
-		(at 265.43 172.72 0)
-		(fields_autoplaced yes)
-		(effects
-			(font
-				(size 1.27 1.27)
-			)
-			(justify left)
-		)
-		(property "Intersheetrefs" "${INTERSHEET_REFS}"
-			(at 274.8257 172.72 0)
-			(hide yes)
-			(show_name no)
-			(do_not_autoplace no)
-			(effects
-				(font
-					(size 1.27 1.27)
-				)
-				(justify left)
-			)
-		)
-	)
-	(global_label "PS_SRST"
-		(shape input)
-		(at 193.04 60.96 180)
-		(fields_autoplaced yes)
-		(effects
-			(font
-				(size 1.27 1.27)
-			)
-			(justify right)
-		)
-		(property "Intersheetrefs" "${INTERSHEET_REFS}"
-			(at 181.9511 60.96 0)
-			(hide yes)
-			(show_name no)
-			(do_not_autoplace no)
-			(effects
-				(font
-					(size 1.27 1.27)
-				)
-				(justify right)
-			)
-		)
-	)
-	(global_label "5V0_IN"
-		(shape input)
-		(at 142.24 171.45 0)
-		(fields_autoplaced yes)
-		(effects
-			(font
-				(size 1.27 1.27)
-			)
-			(justify left)
-		)
-		(property "Intersheetrefs" "${INTERSHEET_REFS}"
-			(at 151.6357 171.45 0)
-			(hide yes)
-			(show_name no)
-			(do_not_autoplace no)
-			(effects
-				(font
-					(size 1.27 1.27)
-				)
-				(justify left)
-			)
-		)
-	)
-	(global_label "GTR_REFCLK0_C2M_N"
-		(shape input)
-		(at 200.66 142.24 180)
-		(fields_autoplaced yes)
-		(effects
-			(font
-				(size 1.27 1.27)
-			)
-			(justify right)
-		)
-		(property "Intersheetrefs" "${INTERSHEET_REFS}"
-			(at 177.7178 142.24 0)
-			(hide yes)
-			(show_name no)
-			(do_not_autoplace no)
-			(effects
-				(font
-					(size 1.27 1.27)
-				)
-				(justify right)
-			)
-		)
-	)
-	(global_label "GTR_REFCLK0_C2M_P"
-		(shape input)
-		(at 200.66 139.7 180)
-		(fields_autoplaced yes)
-		(effects
-			(font
-				(size 1.27 1.27)
-			)
-			(justify right)
-		)
-		(property "Intersheetrefs" "${INTERSHEET_REFS}"
-			(at 177.7783 139.7 0)
+			(at 189.2082 171.45 0)
 			(hide yes)
 			(show_name no)
@@
 				)
 				(justify left)
-			)
-		)
-	)
-	(global_label "5V0_IN"
-		(shape input)
-		(at 58.42 170.18 180)
-		(fields_autoplaced yes)
-		(effects
-			(font
-				(size 1.27 1.27)
-			)
-			(justify right)
-		)
-		(property "Intersheetrefs" "${INTERSHEET_REFS}"
-			(at 49.0243 170.18 0)
-			(hide yes)
-			(show_name no)
-			(do_not_autoplace no)
-			(effects
-				(font
-					(size 1.27 1.27)
-				)
-				(justify right)
 			)
 		)
@@
 			(hide yes)
 			(show_name no)
+			(do_not_autoplace no)
+			(effects
+				(font
+					(size 1.27 1.27)
+				)
+				(justify right)
+			)
+		)
+	)
+	(global_label "5V0_SOM"
+		(shape input)
+		(at 58.42 170.18 180)
+		(fields_autoplaced yes)
+		(effects
+			(font
+				(size 1.27 1.27)
+			)
+			(justify right)
+		)
+		(property "Intersheetrefs" "${INTERSHEET_REFS}"
+			(at 46.9682 170.18 0)
+			(hide yes)
+			(show_name no)

Commit message: update
Other:
- note added: "K26 BOOT MODE SELECT S1-1 = PS_MODE3 S1-2 = PS_MODE2 S1-3 = PS_MODE1 S1-4 = PS_MODE0 SWITCH ON = LOGIC 0 / CONNECTED TO GND SWITCH OFF = LOGIC 1 / SOM INTERNAL 1.8V PULL-UP DEFAULT KV260/QSPI32: 0010 = ON, ON, OFF, ON PS JTAG BOOT: 0000 = ON, ON, ON, ON PRODUCTION eMMC: 0110 = ON, OFF, OFF, ON DIRECT SD1 3.0: 1110 = OFF, OFF, OFF, ON DIRECT SD1 2.0: 0101 = ON, OFF, ON, OFF SET SWITCHES ONLY WHILE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"
Changed lines of the file:
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@@
+		)
+	)
+	(text "K26 BOOT MODE SELECT\n\nS1-1 = PS_MODE3\nS1-2 = PS_MODE2\nS1-3 = PS_MODE1\nS1-4 = PS_MODE0\n\nSWITCH ON  = LOGIC 0 / CONNECTED TO GND\nSWITCH OFF = LOGIC 1 / SOM INTERNAL 1.8V PULL-UP\n\nDEFAULT KV260/QSPI32: 0010 = ON, ON, OFF, ON\nPS JTAG BOOT:         0000 = ON, ON, ON, ON\nPRODUCTION eMMC:      0110 = ON, OFF, OFF, ON\nDIRECT SD1 3.0:       1110 = OFF, OFF, OFF, ON\nDIRECT SD1 2.0:       0101 = ON, OFF, ON, OFF\n\nSET SWITCHES ONLY WHILE POWER IS OFF OR PS_POR_B IS ASSERTED.\nRESERVED MODE SETTINGS MUST NOT BE USED."
+		(exclude_from_sim no)
+		(at -30.226 86.868 0)
+		(effects
+			(font
+				(size 1.27 1.27)
+			)
 		)
 	)

Commit message: update for verification
Parts:
- added TP43: MIO35_PMU_GPO, TestPoint:TestPoint_THTPad_1.5x1.5mm_Drill0.7mm, symbol Connector:TestPoint
Connections:
- net at J10.B28 (MIO35_PMU_GPO): now also TP43.1
- no-connect marks 30 -> 29
Changed lines of the file:
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@@
 	)
 	(no_connect
-		(at 121.92 90.17)
-	)
-	(no_connect
 		(at 214.63 149.86)
 	)
@@
 	(wire
 		(pts
+			(xy 121.92 90.17) (xy 152.4 90.17)
+		)
+		(stroke
+			(width 0)
+			(type default)
+		)
+	)
+	(wire
+		(pts
 			(xy 121.92 54.61) (xy 158.75 54.61)
 		)
@@
 					(unit 1)
 				)
+			)
+		)
+	)
+	(symbol
+		(lib_id "Connector:TestPoint")
+		(at 152.4 90.17 0)
+		(unit 1)
+		(body_style 1)
+		(exclude_from_sim no)
+		(in_bom yes)
+		(on_board yes)
+		(in_pos_files yes)
+		(dnp no)
+		(property "Reference" "TP43"
+			(at 152.908 88.9 0)
+			(show_name no)
+			(do_not_autoplace no)
+			(effects
+				(font
+					(size 1.27 1.27)
+				)
+				(justify left)
+			)
+		)
+		(property "Value" "MIO35_PMU_GPO"
+			(at 135.89 88.9 0)
+			(show_name no)
+			(do_not_autoplace no)
+			(effects
+				(font
+					(size 1.27 1.27)
+				)
+				(justify left)
+			)
+		)
+		(property "Footprint" "TestPoint:TestPoint_THTPad_1.5x1.5mm_Drill0.7mm"
+			(at 157.48 90.17 0)
+			(hide yes)
+			(show_name no)
+			(do_not_autoplace no)
+			(effects
+				(font
+					(size 1.27 1.27)
+				)
+			)
+		)
+		(property "Datasheet" ""
+			(at 157.48 90.17 0)
+			(hide yes)
+			(show_name no)
+			(do_not_autoplace no)
+			(effects
+				(font
+					(size 1.27 1.27)
+				)
+			)
+		)
+		(property "Description" "test point"
+			(at 152.4 90.17 0)
+			(hide yes)
+			(show_name no)
+			(do_not_autoplace no)
+			(effects
+				(font
+					(size 1.27 1.27)
+				)
+			)
+		)
+		(pin "1"
+		)
+		(instances
+			(project "PSEC5_Ctrl_Board"
+				(path "/165f2ae6-d522-4adf-a6c4-bb137b209d33/1f6d7a03-cfad-4370-8d2b-49ab19e248d8"
+					(reference "TP43")
+					(unit 1)
+				)
