File: KADC_CONTROLLER_V2/SD_New.kicad_sch (KiCad schematic)
At the start: 28 parts, among them IC2 NVT4858HKZ, J8 1040310811, U22 TPS22913BYZVT, U23 NX3P1108UKZ, U24 74AUP1G04GW-Q100, U25 NX3P1108UKZ

Commit message: many updates
Parts:
- added C187: 2.2u, Capacitor_SMD:C_0603_1608Metric, symbol Device:C_Small
- added C188: 10u, Capacitor_SMD:C_0603_1608Metric, symbol Device:C_Small
- added C189, C192, C193: 0.1u, Capacitor_SMD:C_0603_1608Metric, symbol Device:C_Small
- added C190, C191: 0.47u, Capacitor_SMD:C_0603_1608Metric, symbol Device:C_Small
- added J9: 5025700893, 502570-0893_MOL, symbol 5025700893:5025700893
- added Q3: FDN336P, symbol Simulation_SPICE:PMOS
- added Q4: DMN2310U-7, Package_TO_SOT_SMD:TSOT-23, symbol Simulation_SPICE:NMOS
- added R164: 4.7k, Resistor_SMD:R_0603_1608Metric, symbol Device:R_Small_US
- added R165, R166, R168: 10k, Resistor_SMD:R_0603_1608Metric, symbol Device:R_Small_US
- added R167: 1k, Resistor_SMD:R_0603_1608Metric, symbol Device:R_Small_US
- added R169, R170, R171, R172, R173, R174: 30R, Resistor_SMD:R_0603_1608Metric, symbol Device:R_Small_US
- added U44: PI4ULS3V4857GEAEX, BGA20_WLCSP_PI4ULS3V4857_DIO, symbol PI4ULS3V4857GEAEX:PI4ULS3V4857GEAEX
Connections:
- net GND: now also C187.2, C188.2, C189.2, C192.2, C193.2, J9.10 (DETECT_SWITCH), Q4.3 (S)
- net SD_CLKA: now also R170.1
- net SD_CMDA: now also R169.1
- net SD_DAT0A: now also R171.1
- net SD_DAT1A: now also R172.1
- net SD_DAT2A: now also R173.1
- net SD_DAT3A: now also R174.1
- net SD_DETECT: now also J9.9 (DETECT_LEVER), R164.1, U44.B2 (CD)
- net SD_SEL: now also U44.E3 (SEL)
- new net: C187.1, R165.1, U44.B3 (VCCB)
- new net: J9.2 (CD/DAT3), R165.2, U44.B4 (DAT3B)
- new net: R173.2, U44.A1 (DAT2A)
- new net: J9.1 (DAT2), U44.A4 (DAT2B)
- new net: R174.2, U44.B1 (DAT3A)
- new net: R169.2, U44.C1 (CMDA)
- new net: J9.3 (CMD), U44.C4 (CMDB)
- new net: R171.2, U44.D1 (DAT0A)
- new net: R170.2, U44.D2 (CLKA)
- new net: J9.5 (CLK), U44.D3 (CLKB)
- new net: J9.7 (DAT0), U44.D4 (DAT0B)
- new net: R172.2, U44.E1 (DAT1A)
- new net: J9.8 (DAT1), U44.E4 (DAT1B)
- new net: C190.2, C191.1, Q3.2 (G), R166.2, R167.1
- new net: C188.1, C189.1, C191.2, J9.4 (VDD), Q3.1 (D)
- new net: Q4.1 (D), R167.2
- new net: Q4.2 (G), R168.2
- new net PS_1V8: C193.1, R164.2, U44.A2 (VCCA)
- new net PS_3V3: C190.1, C192.1, Q3.3 (S), R166.1, R168.1, U44.A3 (VSD)
- no-connect marks 1 -> 2
Other:
- note added: "SD PROPER"
- note added: "SD_RESET_B"
- note added: "This SD Card will be on a breakout board attached via a connector (TBD) This is to avoid large costs with blind vias fro the SD translator since this is the only component on the board that requires blind vias"
- moved on the sheet: C123, C124, C125, C126, C127, C128, C43, C96, IC2, J8, R116, R117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

Commit message: More Things
Parts:
- added C244: 22p, symbol Device:C_Small
- added Q11: DMN2310U-7, Package_TO_SOT_SMD:TSOT-23, symbol Simulation_SPICE:NMOS
Connections:
- net GND: now also C244.2
- net PS_1V8: now also Q11.2 (G)
- net at Q4.2 (G), R168.2: now also C244.1, Q11.1 (D)
- new net PS_POR: Q11.3 (S)

Commit message: quick changes
Parts:
- removed C123, C125, C126, C127, C128, C43: 0.1u, Capacitor_SMD:C_0603_1608Metric, symbol Device:C_Small
- removed C124: 10u, Capacitor_SMD:C_0603_1608Metric, symbol Device:C_Small
- removed C96: 100pF DNP, Capacitor_SMD:C_0603_1608Metric, symbol Device:C_Small
- removed IC2: NVT4858HKZ, NVT4858HKZ, symbol NVT4858HKZ:NVT4858HKZ
- removed J8: 1040310811, 1040310811:104031-0811_MOL, symbol PSEC5_ctrlbd:1040310811
- removed R116, R117, R118, R119, R121, R122: 33.2R, Resistor_SMD:R_0603_1608Metric, symbol Device:R_Small_US
- removed R120, R123, R125: 10k, Resistor_SMD:R_0603_1608Metric, symbol Device:R_Small_US
- removed R124, R126, R127, R128: 0R, Resistor_SMD:R_0603_1608Metric, symbol Device:R_Small_US
- removed R129: 5k, Resistor_SMD:R_0603_1608Metric, symbol Device:R_Small_US
- removed U22: TPS22913BYZVT, TPS22913:TPS22913BYZVT, symbol TPS22913:TPS22913BYZVT
- removed U23, U25: NX3P1108UKZ, NX3P1108:BGA4C50P2X2_97X97X58N, symbol NX3P1108:NX3P1108UKZ
- removed U24: 74AUP1G04GW-Q100, Package_TO_SOT_SMD:SOT-353_SC-70-5, symbol 74AUP1G04GW:74AUP1G04GW-Q100
Connections:
- no-connect marks 2 -> 1
Other:
- note removed: "SD Inputs"
- note removed: "SD Outputs"
- note removed: "SD_CLKA"
- note removed: "SD_SEL SD_DAT0A SD_DAT1A SD_DAT2A SD_DAT3A SD_CMDA"

Commit message: Added footprints, updated schematic
Connections:
- net GND: now also J9.6 (VSS), U44.C2 (GND), U44.C3 (GND)
Changed lines of the file:
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@@
+	)
+	(junction
+		(at 201.93 330.2)
+		(diameter 0)
+		(color 0 0 0 0)
 	)
 	(junction
@@
 	(wire
 		(pts
+			(xy 290.83 332.74) (xy 290.83 340.36)
+		)
+		(stroke
+			(width 0)
+			(type default)
+		)
+	)
+	(wire
+		(pts
 			(xy 224.79 248.92) (xy 207.01 248.92)
 		)
@@
 	(wire
 		(pts
+			(xy 201.93 330.2) (xy 201.93 345.44)
+		)
+		(stroke
+			(width 0)
+			(type default)
+		)
+	)
+	(wire
+		(pts
 			(xy 88.9 322.58) (xy 146.05 322.58)
 		)
@@
 	(wire
 		(pts
+			(xy 191.77 330.2) (xy 201.93 330.2)
+		)
+		(stroke
+			(width 0)
+			(type default)
+		)
+	)
+	(wire
+		(pts
 			(xy 53.34 229.87) (xy 88.9 229.87)
 		)
@@
 	(wire
 		(pts
+			(xy 201.93 327.66) (xy 201.93 330.2)
+		)
+		(stroke
+			(width 0)
+			(type default)
+		)
+	)
+	(wire
+		(pts
 			(xy 179.07 267.97) (xy 175.26 267.97)
 		)
@@
 		(pts
 			(xy 260.35 278.13) (xy 260.35 281.94)
+		)
+		(stroke
+			(width 0)
+			(type default)
+		)
+	)
+	(wire
+		(pts
+			(xy 191.77 327.66) (xy 201.93 327.66)
 		)
 		(stroke
@@
 	)
 	(symbol
+		(lib_id "power:GND")
+		(at 290.83 340.36 0)
+		(unit 1)
+		(body_style 1)
+		(exclude_from_sim no)
+		(in_bom yes)
+		(on_board yes)
+		(in_pos_files yes)
+		(dnp no)
+		(fields_autoplaced yes)
+		(property "Reference" "#PWR041"
+			(at 290.83 346.71 0)
+			(hide yes)
+			(show_name no)
+			(do_not_autoplace no)
+			(effects
+				(font
+					(size 1.27 1.27)
+				)
+			)
+		)
+		(property "Value" "GND"
+			(at 290.83 345.44 0)
+			(show_name no)
+			(do_not_autoplace no)
+			(effects
+				(font
+					(size 1.27 1.27)
+				)
+			)
+		)
+		(property "Footprint" ""
+			(at 290.83 340.36 0)
+			(hide yes)
+			(show_name no)
+			(do_not_autoplace no)
+			(effects
+				(font
+					(size 1.27 1.27)
+				)
+			)
+		)
+		(property "Datasheet" ""
+			(at 290.83 340.36 0)
+			(hide yes)
+			(show_name no)
+			(do_not_autoplace no)
+			(effects
+				(font
+					(size 1.27 1.27)
+				)
+			)
+		)
+		(property "Description" "Power symbol creates a global label with name \"GND\" , ground"
+			(at 290.83 340.36 0)
+			(hide yes)
+			(show_name no)
+			(do_not_autoplace no)
+			(effects
+				(font
+					(size 1.27 1.27)
+				)
+			)
+		)
+		(pin "1"
+		)
+		(instances
+			(project "PSEC5_Ctrl_Board"
+				(path "/165f2ae6-d522-4adf-a6c4-bb137b209d33/1f6d7a03-cfad-4370-8d2b-49ab19e248d8/15f57d5c-54b3-4ba8-a361-8040b738c0f2"
+					(reference "#PWR041")
+					(unit 1)
+				)
+			)
+		)
+	)
+	(symbol
 		(lib_id "Device:R_Small_US")
 		(at 86.36 314.96 90)
@@
 					(unit 1)
 				)
+			)
+		)
+	)
+	(symbol
+		(lib_id "power:GND")
+		(at 201.93 345.44 0)
+		(unit 1)
+		(body_style 1)
+		(exclude_from_sim no)
+		(in_bom yes)
+		(on_board yes)
+		(in_pos_files yes)
+		(dnp no)
+		(fields_autoplaced yes)
+		(property "Reference" "#PWR040"
+			(at 201.93 351.79 0)
+			(hide yes)
+			(show_name no)
+			(do_not_autoplace no)
+			(effects
+				(font
+					(size 1.27 1.27)
+				)
+			)
+		)
+		(property "Value" "GND"
+			(at 201.93 350.52 0)
+			(show_name no)
+			(do_not_autoplace no)
+			(effects
+				(font
+					(size 1.27 1.27)
+				)
+			)
+		)
+		(property "Footprint" ""
+			(at 201.93 345.44 0)
+			(hide yes)
+			(show_name no)
+			(do_not_autoplace no)
+			(effects
+				(font
+					(size 1.27 1.27)
+				)
+			)
+		)
+		(property "Datasheet" ""
+			(at 201.93 345.44 0)
+			(hide yes)
+			(show_name no)
+			(do_not_autoplace no)
+			(effects
+				(font
+					(size 1.27 1.27)
+				)
+			)
+		)
+		(property "Description" "Power symbol creates a global label with name \"GND\" , ground"
+			(at 201.93 345.44 0)
+			(hide yes)
+			(show_name no)
+			(do_not_autoplace no)
+			(effects
+				(font
+					(size 1.27 1.27)
+				)
+			)
+		)
+		(pin "1"
+		)
+		(instances
+			(project "PSEC5_Ctrl_Board"
+				(path "/165f2ae6-d522-4adf-a6c4-bb137b209d33/1f6d7a03-cfad-4370-8d2b-49ab19e248d8/15f57d5c-54b3-4ba8-a361-8040b738c0f2"
+					(reference "#PWR040")
+					(unit 1)
+				)

Commit message: Reupdate for verify
Parts:
- J9: footprint 502570-0893_MOL -> 5025700893:502570-0893_MOL
- U44: footprint BGA20_WLCSP_PI4ULS3V4857_DIO -> PI4ULS3V4857GEAEX:BGA20_WLCSP_PI4ULS3V4857_DIO
Changed lines of the file:
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@@
 			)
 		)
-		(property "Footprint" "BGA20_WLCSP_PI4ULS3V4857_DIO"
+		(property "Footprint" "PI4ULS3V4857GEAEX:BGA20_WLCSP_PI4ULS3V4857_DIO"
 			(at 166.116 281.178 0)
 			(hide yes)
@@
 			)
 		)
-		(property "Footprint" "502570-0893_MOL"
+		(property "Footprint" "5025700893:502570-0893_MOL"
 			(at 290.068 281.178 0)
 			(hide yes)

Commit message: changes for check
Parts:
- removed Q11, Q4: DMN2310U-7, Package_TO_SOT_SMD:TSOT-23, symbol Simulation_SPICE:NMOS
- added Q15, Q19: BSS806NEH6327XTSA1, Package_TO_SOT_SMD:SOT-23-3, symbol Transistor_FET:Q_NMOS_GSD
- C244: footprint (none) -> Capacitor_SMD:C_0603_1608Metric
- Q3: footprint (none) -> FDN336P:SOT23-3_527AG_FAS
Connections:
- net GND: now also Q15.2 (S)
- net PS_1V8: now also Q19.1 (G)
- net PS_POR: now also Q19.2 (S)
- net at R167.2: now also Q15.3 (D)
- net at C244.1, R168.2: now also Q15.1 (G), Q19.3 (D)
Other:
- moved on the sheet: C244
